File: Urbie/wiring-diagram/RearLights.sch (KiCad schematic (older format))
At the start: 13 parts

Commit message: I don't know what changed
Parts:
- L? (x5): symbol Lamp -> Lamp-RESCUE-Version1
Connections:
- new net: L?.~, L?.~, L?.~, P?.4 (P4)
Changed lines of the file:
@@
 EESchema Schematic File Version 2
+LIBS:Version1-rescue
 LIBS:power
 LIBS:device
@@
 $EndDescr
 $Comp
-L Lamp L?
+L Lamp-RESCUE-Version1 L?
 U 1 1 587A5960
 P 4075 6950
@@
 $EndComp
 $Comp
-L Lamp L?
+L Lamp-RESCUE-Version1 L?
 U 1 1 587A59FA
 P 4075 6600
@@
 $EndComp
 $Comp
-L Lamp L?
+L Lamp-RESCUE-Version1 L?
 U 1 1 587A5D31
 P 4075 6275
@@
 $EndComp
 $Comp
-L Lamp L?
+L Lamp-RESCUE-Version1 L?
 U 1 1 587A5D8F
 P 4075 5825
@@
 $EndComp
 $Comp
-L Lamp L?
+L Lamp-RESCUE-Version1 L?
 U 1 1 587A5DE7
 P 4100 7425
