File: current_sensor/CanController.sch (KiCad schematic (older format))
At the start: 57 parts, among them P10 CONN_02X03, P11 CONN_02X03, P12 CONN_02X03, P7 CONN_01X03, P8 USB, P9 Term, SW1 RESET, SW2 BOOT, U6 STM32F042C6, U7 mcp2562

Commit message: updated Current Sensor board with changes made to CanSensor (zener diodes)
Parts:
- removed D3, D5, D7: D_Schottky_Small, Diodes_SMD:SOD-123, symbol D_Schottky_Small
- D1, D2: symbol Led_Small -> LED_Small
- renumbered D4 to D3, D6 to D4, D8 to D5
Other:
- moved on the sheet: P8, R7
Changed lines of the file:
@@
 EESchema Schematic File Version 2
+LIBS:Current Sensor-rescue
 LIBS:power
 LIBS:device
@@
 CAN_L
 $Comp
-L Led_Small D1
+L LED_Small D1
 U 1 1 581EFCE8
 P 9600 3350
@@
 $EndComp
 $Comp
-L Led_Small D2
+L LED_Small D2
 U 1 1 581EFCE9
 P 9600 3650
@@
 L USB_OTG P8
 U 1 1 581EFCEC
-P 1100 7000
+P 900 7050
 AR Path="/581EFCEC" Ref="P8"  Part="1"
 AR Path="/581EF7A1/581EFCEC" Ref="P8"  Part="1"
-F 0 "P8" V 800 7000 50  0000 C CNN
-F 1 "USB" H 1100 7200 50  0000 C CNN
-F 2 "Connect:USB_Micro-B" H 1050 6900 50  0001 C CNN
-F 3 "" V 1050 6900 50  0000 C CNN
-F 4 "Mouser" V 1100 7000 60  0001 C CNN "Distributor"
-F 5 "649-10118194-0001LF" V 1100 7000 60  0001 C CNN "PN"
-	1    1100 7000
-	0    -1   1    0
-$EndComp
-Text Label 1500 6900 0    60   ~ 0
+F 0 "P8" V 600 7050 50  0000 C CNN
+F 1 "USB" H 750 7400 50  0000 C CNN
+F 2 "Connect:USB_Micro-B" H 850 6950 50  0001 C CNN
+F 3 "" V 850 6950 50  0000 C CNN
+F 4 "Mouser" V 900 7050 60  0001 C CNN "Distributor"
+F 5 "649-10118194-0001LF" V 900 7050 60  0001 C CNN "PN"
+	1    900  7050
+	1    0    0    -1
+$EndComp
+Text Label 1300 7150 0    60   ~ 0
 USB_DM
-Text Label 1500 7000 0    60   ~ 0
+Text Label 1300 7050 0    60   ~ 0
 USB_DP
 $Comp
 L +5V #PWR033
 U 1 1 581EFCED
-P 1450 6750
-F 0 "#PWR033" H 1450 6600 50  0001 C CNN
-F 1 "+5V" H 1450 6890 50  0000 C CNN
-F 2 "" H 1450 6750 50  0000 C CNN
-F 3 "" H 1450 6750 50  0000 C CNN
-	1    1450 6750
+P 1250 6800
+F 0 "#PWR033" H 1250 6650 50  0001 C CNN
+F 1 "+5V" H 1250 6940 50  0000 C CNN
+F 2 "" H 1250 6800 50  0000 C CNN
+F 3 "" H 1250 6800 50  0000 C CNN
+	1    1250 6800
 	1    0    0    -1
 $EndComp
@@
 L GND #PWR034
 U 1 1 581EFCEE
-P 1400 7500
-F 0 "#PWR034" H 1400 7250 50  0001 C CNN
-F 1 "GND" H 1400 7350 50  0000 C CNN
-F 2 "" H 1400 7500 50  0000 C CNN
-F 3 "" H 1400 7500 50  0000 C CNN
-	1    1400 7500
+P 1000 7650
+F 0 "#PWR034" H 1000 7400 50  0001 C CNN
+F 1 "GND" H 1000 7500 50  0000 C CNN
+F 2 "" H 1000 7650 50  0000 C CNN
+F 3 "" H 1000 7650 50  0000 C CNN
+	1    1000 7650
 	1    0    0    -1
 $EndComp
@@
 L R R7
 U 1 1 581EFCF8
-P 1600 7250
-F 0 "R7" V 1680 7250 50  0000 C CNN
-F 1 "100K" V 1600 7250 50  0000 C CNN
-F 2 "Resistors_SMD:R_0603_HandSoldering" H 1530 7250 50  0001 C CNN
-F 3 "" H 1600 7250 50  0000 C CNN
-F 4 "Mouser" V 1600 7250 60  0001 C CNN "Distributor"
-F 5 "71-CRCW0603-100K-E3" V 1600 7250 60  0001 C CNN "PN"
-	1    1600 7250
+P 1300 7400
+F 0 "R7" V 1380 7400 50  0000 C CNN
+F 1 "100K" V 1300 7400 50  0000 C CNN
+F 2 "Resistors_SMD:R_0603_HandSoldering" H 1230 7400 50  0001 C CNN
+F 3 "" H 1300 7400 50  0000 C CNN
+F 4 "Mouser" V 1300 7400 60  0001 C CNN "Distributor"
+F 5 "71-CRCW0603-100K-E3" V 1300 7400 60  0001 C CNN "PN"
+	1    1300 7400
 	1    0    0    -1
 $EndComp
@@
 $EndComp
 $Comp
-L D_Schottky_Small D4
+L D_Schottky_Small D3
 U 1 1 582A2F6F
 P 2600 1950
-F 0 "D4" H 2550 2030 50  0000 L CNN
+F 0 "D3" H 2550 2030 50  0000 L CNN
 F 1 "D_Schottky_Small" H 2320 1870 50  0001 L CNN
 F 2 "Diodes_SMD:SOD-123" V 2600 1950 50  0001 C CNN
@@
 	0    1    1    0
 $EndComp
-$Comp
-L D_Schottky_Small D3
-U 1 1 582A322E
-P 2600 1350
-F 0 "D3" H 2550 1430 50  0000 L CNN
-F 1 "D_Schottky_Small" H 2320 1270 50  0001 L CNN
-F 2 "Diodes_SMD:SOD-123" V 2600 1350 50  0001 C CNN
-F 3 "" V 2600 1350 50  0000 C CNN
-F 4 "Mouser" H 2600 1350 60  0001 C CNN "Distributor"
-F 5 "512-SS14FL " H 2600 1350 60  0001 C CNN "PN"
-	1    2600 1350
-	0    1    1    0
-$EndComp
-$Comp
-L D_Schottky_Small D5
-U 1 1 582A34E4
-P 2600 2850
-F 0 "D5" H 2550 2930 50  0000 L CNN
-F 1 "D_Schottky_Small" H 2320 2770 50  0001 L CNN
-F 2 "Diodes_SMD:SOD-123" V 2600 2850 50  0001 C CNN
-F 3 "" V 2600 2850 50  0000 C CNN
-F 4 "Mouser" H 2600 2850 60  0001 C CNN "Distributor"
-F 5 "512-SS14FL " H 2600 2850 60  0001 C CNN "PN"
-	1    2600 2850
-	0    1    1    0
-$EndComp
 Wire Wire Line
 	6450 2350 6450 2550
@@
 	7350 1900 7400 1900
 Wire Wire Line
-	1500 7000 1400 7000
-Wire Wire Line
-	1500 6900 1400 6900
-Wire Wire Line
-	1450 6750 1450 6800
-Wire Wire Line
-	1450 6800 1400 6800
-Wire Wire Line
-	1400 7200 1400 7500
-Wire Wire Line
-	1000 7400 1600 7400
-Connection ~ 1400 7400
-Wire Wire Line
-	1400 7100 1600 7100
+	1300 7050 1200 7050
+Wire Wire Line
+	1300 7150 1200 7150
+Wire Wire Line
+	1250 6800 1250 6850
+Wire Wire Line
+	1250 6850 1200 6850
 Wire Wire Line
 	6350 5900 6350 6050
@@
 Wire Wire Line
 	4450 3900 4950 3900
-$Comp
-L D_Schottky_Small D7
-U 1 1 582A3825
-P 2550 4450
-F 0 "D7" H 2500 4530 50  0000 L CNN
-F 1 "D_Schottky_Small" H 2270 4370 50  0001 L CNN
-F 2 "Diodes_SMD:SOD-123" V 2550 4450 50  0001 C CNN
-F 3 "" V 2550 4450 50  0000 C CNN
-F 4 "Mouser" H 2550 4450 60  0001 C CNN "Distributor"
-F 5 "512-SS14FL " H 2550 4450 60  0001 C CNN "PN"
-	1    2550 4450
-	0    1    1    0
-$EndComp
 $Comp
 L CONN_02X03 P10
@@
 	4450 3300 4950 3300
 $Comp
-L +3.3V #PWR045
-U 1 1 582A86B9
-P 2600 1200
-F 0 "#PWR045" H 2600 1050 50  0001 C CNN
-F 1 "+3.3V" H 2600 1340 50  0000 C CNN
-F 2 "" H 2600 1200 50  0000 C CNN
-F 3 "" H 2600 1200 50  0000 C CNN
-	1    2600 1200
-	1    0    0    -1
-$EndComp
-$Comp
-L GND #PWR046
+L GND #PWR045
 U 1 1 582A8E96
 P 2600 2100
-F 0 "#PWR046" H 2600 1850 50  0001 C CNN
+F 0 "#PWR045" H 2600 1850 50  0001 C CNN
 F 1 "GND" H 2600 1950 50  0000 C CNN
 F 2 "" H 2600 2100 50  0000 C CNN
@@
 $EndComp
 $Comp
-L GND #PWR047
+L GND #PWR046
 U 1 1 583A28CD
 P 1400 3700
-F 0 "#PWR047" H 1400 3450 50  0001 C CNN
+F 0 "#PWR046" H 1400 3450 50  0001 C CNN
 F 1 "GND" H 1400 3550 50  0000 C CNN
 F 2 "" H 1400 3700 50  0000 C CNN
@@
 $EndComp
 $Comp
-L +3.3V #PWR048
-U 1 1 583A2921
-P 2600 2700
-F 0 "#PWR048" H 2600 2550 50  0001 C CNN
-F 1 "+3.3V" H 2600 2840 50  0000 C CNN
-F 2 "" H 2600 2700 50  0000 C CNN
-F 3 "" H 2600 2700 50  0000 C CNN
-	1    2600 2700
-	1    0    0    -1
-$EndComp
-$Comp
-L GND #PWR049
+L GND #PWR047
 U 1 1 583A2935
 P 2600 3600
-F 0 "#PWR049" H 2600 3350 50  0001 C CNN
+F 0 "#PWR047" H 2600 3350 50  0001 C CNN
 F 1 "GND" H 2600 3450 50  0000 C CNN
 F 2 "" H 2600 3600 50  0000 C CNN
@@
 $EndComp
 $Comp
-L GND #PWR050
+L GND #PWR048
 U 1 1 583A78B2
 P 1400 5300
-F 0 "#PWR050" H 1400 5050 50  0001 C CNN
+F 0 "#PWR048" H 1400 5050 50  0001 C CNN
 F 1 "GND" H 1400 5150 50  0000 C CNN
 F 2 "" H 1400 5300 50  0000 C CNN
@@
 $EndComp
 $Comp
-L +3.3V #PWR051
-U 1 1 583A7906
-P 2550 4300
-F 0 "#PWR051" H 2550 4150 50  0001 C CNN
-F 1 "+3.3V" H 2550 4440 50  0000 C CNN
-F 2 "" H 2550 4300 50  0000 C CNN
-F 3 "" H 2550 4300 50  0000 C CNN
-	1    2550 4300
-	1    0    0    -1
-$EndComp
-$Comp
-L GND #PWR052
+L GND #PWR049
 U 1 1 583A791A
 P 2550 5200
-F 0 "#PWR052" H 2550 4950 50  0001 C CNN
+F 0 "#PWR049" H 2550 4950 50  0001 C CNN
 F 1 "GND" H 2550 5050 50  0000 C CNN
 F 2 "" H 2550 5200 50  0000 C CNN
@@
 Connection ~ 1100 1150
 $Comp
-L D_Schottky_Small D6
+L D_Schottky_Small D4
 U 1 1 582A32BC
 P 2600 3450
-F 0 "D6" H 2550 3530 50  0000 L CNN
+F 0 "D4" H 2550 3530 50  0000 L CNN
 F 1 "D_Schottky_Small" H 2320 3370 50  0001 L CNN
 F 2 "Diodes_SMD:SOD-123" V 2600 3450 50  0001 C CNN
@@
 $EndComp
 $Comp
-L D_Schottky_Small D8
+L D_Schottky_Small D5
 U 1 1 582A35CA
 P 2550 5050
-F 0 "D8" H 2500 5130 50  0000 L CNN
+F 0 "D5" H 2500 5130 50  0000 L CNN
 F 1 "D_Schottky_Small" H 2270 4970 50  0001 L CNN
 F 2 "Diodes_SMD:SOD-123" V 2550 5050 50  0001 C CNN
@@
 	2500 4750 2850 4750
 Wire Wire Line
-	2550 4300 2550 4350
-Wire Wire Line
 	2550 5200 2550 5150
 Wire Wire Line
 	2550 4850 2500 4850
-Wire Wire Line
-	2550 4550 2550 4950
 Connection ~ 2550 4750
 Wire Wire Line
 	2500 4650 2550 4650
 Connection ~ 2550 4850
-Connection ~ 2550 4650
 Wire Wire Line
 	1000 4250 1700 4250
 Connection ~ 1100 4250
 Connection ~ 1400 4250
-Wire Wire Line
-	2600 2950 2600 3350
 Connection ~ 2600 3250
-Connection ~ 2600 3050
 Connection ~ 2600 3150
 Text Label 2850 3150 2    60   ~ 0
 V2a
 Wire Wire Line
-	2600 2750 2600 2700
-Wire Wire Line
 	2600 3600 2600 3550
 Wire Wire Line
@@
 Connection ~ 1400 2650
 Wire Wire Line
-	2600 1450 2600 1850
-Wire Wire Line
 	2500 1550 2600 1550
-Connection ~ 2600 1550
 Wire Wire Line
 	2500 1650 2850 1650
@@
 Wire Wire Line
 	2600 2050 2600 2100
-Wire Wire Line
-	2600 1250 2600 1200
 Text Notes 8500 800  0    60   ~ 0
 CAN tranciver
@@
 	7025 5700 6750 5700
 $Comp
-L GND #PWR053
+L GND #PWR050
 U 1 1 58806A24
 P 8000 5025
-F 0 "#PWR053" H 8000 4775 50  0001 C CNN
+F 0 "#PWR050" H 8000 4775 50  0001 C CNN
 F 1 "GND" H 8000 4875 50  0000 C CNN
 F 2 "" H 8000 5025 50  0000 C CNN
@@
 Wire Wire Line
 	8000 4950 7650 4950
+Wire Wire Line
+	1200 7250 1300 7250
+Wire Wire Line
+	800  7450 800  7600
+Wire Wire Line
+	800  7600 1300 7600
+Wire Wire Line
+	1300 7600 1300 7550
+Wire Wire Line
+	900  7450 900  7600
+Connection ~ 900  7600
+Wire Wire Line
+	1000 7650 1000 7600
+Connection ~ 1000 7600
+Wire Wire Line
+	2600 1550 2600 1850
+Wire Wire Line
+	2600 3050 2600 3350
+Wire Wire Line
+	2550 4650 2550 4950
 $EndSCHEMATC
