File: Urbie/schematics/Engine.sch (KiCad schematic (older format))
At the start: 47 parts

Commit message: added DPDT switch for Hazard lights on Urbie
Parts:
- F?: symbol Fuse -> FUSE
- TH? (x2): symbol Thermistor -> THERMISTOR
Changed lines of the file:
@@
 EESchema Schematic File Version 2
-LIBS:Version1-rescue
+LIBS:UrbieSchematics-rescue
 LIBS:power
 LIBS:device
@@
 LIBS:valves
 LIBS:Supermileage
-LIBS:relays_switches
-LIBS:supermileage
-LIBS:supermileage_computers
-LIBS:switch_dpst
-LIBS:Version1-cache
+LIBS:UrbieSchematics-cache
 EELAYER 25 0
 EELAYER END
@@
 $EndComp
 $Comp
-L Fuse F?
+L FUSE F?
 U 1 1 587B9877
 P 6225 2275
@@
 	5450 5875 5525 5875
 $Comp
-L Thermistor TH?
+L THERMISTOR TH?
 U 1 1 587B9886
 P 2950 5325
@@
 $EndComp
 $Comp
-L Thermistor TH?
+L THERMISTOR TH?
 U 1 1 587B9887
 P 2950 5875
