File: Urbie/schematics/Lights.sch (KiCad schematic (older format))
At the start: 34 parts

Commit message: cleaning up schematics
Parts:
- SW?: symbol UrbieLightSwitch -> UrbieLightSwitch-RESCUE-UrbieSchematics
Changed lines of the file:
@@
 EESchema Schematic File Version 2
+LIBS:UrbieSchematics-rescue
 LIBS:power
 LIBS:device
@@
 Running Lights
 $Comp
-L UrbieLightSwitch SW?
+L UrbieLightSwitch-RESCUE-UrbieSchematics SW?
 U 1 1 58434A5C
 P 3250 6250

Commit message: added DPDT switch for Hazard lights on Urbie
Parts:
- Brights_Indicator, D? (x2): symbol LED -> LED-RESCUE-UrbieSchematics
Changed lines of the file:
@@
 LIBS:Supermileage
 LIBS:UrbieSchematics-cache
-LIBS:EFI_Breakout-cache
 EELAYER 25 0
 EELAYER END
@@
 $EndComp
 $Comp
-L LED Brights_Indicator
+L LED-RESCUE-UrbieSchematics Brights_Indicator
 U 1 1 5827AE7F
 P 6100 6900
@@
 $EndComp
 $Comp
-L LED D?
+L LED-RESCUE-UrbieSchematics D?
 U 1 1 582A8B64
 P 5850 3100
@@
 Connection ~ 7400 3100
 $Comp
-L LED D?
+L LED-RESCUE-UrbieSchematics D?
 U 1 1 582A8E65
 P 5850 1150
