File: Urbie/schematics/SwitchPanel.sch (KiCad schematic (older format))
At the start: 21 parts

Commit message: added DPDT switch for Hazard lights on Urbie
Parts:
- removed SW?: Switch_DPST, symbol Switch_DPST
Connections:
- wire segments 138 -> 136
Other:
- moved on the sheet: CB1, CB2, CB3, CB4
