File: EFI_BREAKOUT/_autosave-efi_backup.kicad_pcb (KiCad board)
At the start: 2 copper layers, 86.1 x 70.1 mm, 56 parts, among them J1 DB25, J10 TEST_1P, J11 TEST_1P, J12 TEST_1P, J13 TEST_1P, J14 TEST_1P, J15 TEST_1P, J16 TEST_1P, J17 TEST_1P, J18 TEST_1P, J19 TEST_1P, J2 TEST_1P, J20 TEST_1P, J21 TEST_1P, J22 TEST_1P, J23 TEST_1P, J24 TEST_1P, J25 TEST_1P, J26 TEST_1P, J27 TEST_1P, J28 TEST_1P, J29 TEST_1P, J3 TEST_1P, J30 TEST_1P, J31 TEST_1P, J32 TEST_1P, J33 TEST_1P, J34 TEST_1P, J35 TEST_1P, J36 TEST_1P, J37 TEST_1P, J38 O2, J39 CANH, J4 TEST_1P, J40 CANL, J41 INJ, J42 TPS, J43 MAT, J44 CLT, J45 TACH, J46 TPS_5V, J5 TEST_1P, J6 TEST_1P, J7 TEST_1P, J8 TEST_1P, J9 TEST_1P, P10 Intake Air Temp, P12 Injector, P13 Coolant Temp, P15 Ignition, P2 CAN, P4 Power, P5 Throttle Position Sensor, P7 O2 Sensor, P9 RPM

Commit message: Final Formatting for production
Edited text and added labeles.
Added power and ground on the test area.
Updated authors and year.
Other:
- board text added: "Megasuirt 2 Breakout Box v2.0 Spring 2018 Sam Ellicott Andrew Ashley Tineka Witt"
- board text removed: "Megasuirt 2 Breakout Box v1.0 Spring 2017 Andy Reigns Sam Ellicott"
Changed lines of the file:
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@@
   (module supermileage_footprints:Molex-UltraFit-2p (layer F.Cu)
     (at 259.08 55.88 90)
-    (fp_text reference P13 (at 0.1016 3.3528 90) (layer F.SilkS)
+    (fp_text reference P13 (at 0.1016 3.3528 90) (layer F.Fab)
       (effects (font (size 1 1) (thickness 0.15)))
     )
@@
   (module supermileage_footprints:Molex-UltraFit-2p (layer F.Cu)
     (at 259.08 66.04 90)
-    (fp_text reference P10 (at 0.1016 3.3528 90) (layer F.SilkS)
+    (fp_text reference P10 (at 0.1016 3.3528 90) (layer F.Fab)
       (effects (font (size 1 1) (thickness 0.15)))
     )
@@
   (module supermileage_footprints:Molex-UltraFit-2p (layer F.Cu)
     (at 201.93 87.63)
-    (fp_text reference P15 (at 0.1016 3.3528) (layer F.SilkS)
+    (fp_text reference P15 (at 0.1016 3.3528) (layer F.Fab)
       (effects (font (size 1 1) (thickness 0.15)))
     )
@@
   (module supermileage_footprints:Molex-UltraFit-2p (layer F.Cu)
     (at 210.83 87.63)
-    (fp_text reference P12 (at 0.1016 3.3528) (layer F.SilkS)
+    (fp_text reference P12 (at 0.1016 3.3528) (layer F.Fab)
       (effects (font (size 1 1) (thickness 0.15)))
     )
@@
   (module supermileage_footprints:Molex-UltraFit-4p (layer F.Cu)
     (at 215.72 74.7)
-    (fp_text reference P9 (at 3.81 -1.27) (layer F.SilkS)
+    (fp_text reference P9 (at 3.81 -1.27) (layer F.Fab)
       (effects (font (size 1 1) (thickness 0.15)))
     )
@@
   (module supermileage_footprints:Molex-UltraFit-4p (layer F.Cu)
     (at 233.5 74.7)
-    (fp_text reference P7 (at 3.81 -1.27) (layer F.SilkS)
+    (fp_text reference P7 (at 3.81 -1.27) (layer F.Fab)
       (effects (font (size 1 1) (thickness 0.15)))
     )
@@
   (module supermileage_footprints:Molex-UltraFit-4p (layer F.Cu)
     (at 189.05 74.7)
-    (fp_text reference P4 (at 3.81 -1.27) (layer F.SilkS)
+    (fp_text reference P4 (at 3.81 -1.27) (layer F.Fab)
       (effects (font (size 1 1) (thickness 0.15)))
     )
@@
     (effects (font (size 1.5 1.5) (thickness 0.3)))
   )
-  (gr_text "Megasuirt 2 Breakout Box v1.0\nSpring 2017\nAndy Reigns\nSam Ellicott\n" (at 185.166 62.738) (layer F.SilkS)
+  (gr_text "Megasuirt 2 Breakout Box v2.0\nSpring 2018\nSam Ellicott\nAndrew Ashley\nTineka Witt" (at 185.166 62.738) (layer F.SilkS)
     (effects (font (size 1.143 1.143) (thickness 0.1905)) (justify left))
   )
