File: Kark/Schematics/EFI_Breakout.sch (KiCad schematic (older format))
At the start: 23 parts, among them J201 DB25, J202 DB25, J203 Megasquirt, P201 CAN, P202 CAN, P203 Power, P204 Power, P205 Throttle Position Sensor, P206 Throttle Position Sensor, P207 O2 Sensor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

Commit message: Removed EFI system and CAN based control from the Karch schematics
Parts:
- J201: symbol DB25_Female -> KarkSchematics-rescue:DB25_Female
- J202: symbol DB25_Male -> KarkSchematics-rescue:DB25_Male
- J203: symbol DB37_Female -> KarkSchematics-rescue:DB37_Female
- P201, P202, P203, P204, P205, P206, P207, P208, P209, P210, P219, P220: symbol CONN_01X04 -> KarkSchematics-rescue:CONN_01X04
- P211, P212, P213, P214, P215, P216, P217, P218: symbol CONN_01X02 -> KarkSchematics-rescue:CONN_01X02
Changed lines of the file:
@@
-EESchema Schematic File Version 2
-LIBS:KarkSchematics-rescue
-LIBS:power
-LIBS:device
-LIBS:switches
-LIBS:relays
-LIBS:motors
-LIBS:transistors
-LIBS:conn
-LIBS:linear
-LIBS:regul
-LIBS:74xx
-LIBS:cmos4000
-LIBS:adc-dac
-LIBS:memory
-LIBS:xilinx
-LIBS:microcontrollers
-LIBS:dsp
-LIBS:microchip
-LIBS:analog_switches
-LIBS:motorola
-LIBS:texas
-LIBS:intel
-LIBS:audio
-LIBS:interface
-LIBS:digital-audio
-LIBS:philips
-LIBS:display
-LIBS:cypress
-LIBS:siliconi
-LIBS:opto
-LIBS:atmel
-LIBS:contrib
-LIBS:valves
-LIBS:relays_switches
-LIBS:supermileage
-LIBS:supermileage_computers
-LIBS:supermileage_sensors
-LIBS:EllicottMicrocontrollers
-LIBS:EllicottInterface
-LIBS:EllicottDisplay
-LIBS:EllicottMisc
-LIBS:EllicottPower
+EESchema Schematic File Version 4
 LIBS:KarkSchematics-cache
-EELAYER 25 0
+EELAYER 29 0
 EELAYER END
 $Descr USLetter 11000 8500
 encoding utf-8
-Sheet 2 10
-Title "EFI Breakout"
+Sheet 2 6
+Title "Kark - Gasoline Prototype"
 Date "2017-01-04"
-Rev "1.0"
-Comp "Cedarville University"
-Comment1 "Edited by Samuel Ellicott"
-Comment2 "Andy Raines"
+Rev "1.1"
+Comp "Cedarville Supermileage"
+Comment1 "Tineka Witt"
+Comment2 "Samuel Ellicott"
 Comment3 "Shematic for Megasquirt breakout box"
 Comment4 ""
 $EndDescr
 $Comp
-L DB25_Female J201
+L KarkSchematics-rescue:DB25_Female J201
 U 1 1 5AB7502A
 P 5275 3450
@@
 O2_3_Sen
 $Comp
-L CONN_01X04 P208
+L KarkSchematics-rescue:CONN_01X04 P208
 U 1 1 5AB7502B
 P 2375 2050
@@
 $EndComp
 $Comp
-L CONN_01X02 P214
+L KarkSchematics-rescue:CONN_01X02 P214
 U 1 1 5AB7502C
 P 3525 2050
@@
 $EndComp
 $Comp
-L CONN_01X02 P218
+L KarkSchematics-rescue:CONN_01X02 P218
 U 1 1 5AB7502D
 P 3975 2050
@@
 $EndComp
 $Comp
-L CONN_01X04 P210
+L KarkSchematics-rescue:CONN_01X04 P210
 U 1 1 5AB7502E
 P 2975 2050
@@
 $EndComp
 $Comp
-L CONN_01X04 P204
+L KarkSchematics-rescue:CONN_01X04 P204
 U 1 1 5AB7502F
 P 1775 2050
@@
 O2_1_GND
 $Comp
-L DB25_Male J202
+L KarkSchematics-rescue:DB25_Male J202
 U 1 1 5AB75030
 P 5925 3450
@@
 $EndComp
 $Comp
-L DB37_Female J203
+L KarkSchematics-rescue:DB37_Female J203
 U 1 1 5AB75031
 P 9775 3400
@@
 CLT_2_B
 $Comp
-L CONN_01X04 P205
+L KarkSchematics-rescue:CONN_01X04 P205
 U 1 1 5AB75032
 P 2275 6500
@@
 $EndComp
 $Comp
-L CONN_01X04 P219
+L KarkSchematics-rescue:CONN_01X04 P219
 U 1 1 5AB75033
 P 4425 6500
@@
 IAC_4_2B
 $Comp
-L CONN_01X02 P211
+L KarkSchematics-rescue:CONN_01X02 P211
 U 1 1 5AB75034
 P 3125 6500
@@
 $EndComp
 $Comp
-L CONN_01X02 P215
+L KarkSchematics-rescue:CONN_01X02 P215
 U 1 1 5AB75035
 P 3725 6500
@@
 	8975 4500 9075 4600
 $Comp
-L CONN_01X04 P202
+L KarkSchematics-rescue:CONN_01X04 P202
 U 1 1 5AB75036
 P 1125 2050
@@
 CAN_4_PWR
 $Comp
-L CONN_01X04 P201
+L KarkSchematics-rescue:CONN_01X04 P201
 U 1 1 5AB75037
 P 1125 1675
@@
 $EndComp
 $Comp
-L CONN_01X04 P203
+L KarkSchematics-rescue:CONN_01X04 P203
 U 1 1 5AB75038
 P 1775 1675
@@
 P_1_GND
 $Comp
-L CONN_01X04 P207
+L KarkSchematics-rescue:CONN_01X04 P207
 U 1 1 5AB75039
 P 2375 1675
@@
 	2325 2250 2325 2350
 $Comp
-L CONN_01X04 P209
+L KarkSchematics-rescue:CONN_01X04 P209
 U 1 1 5AB7503A
 P 2975 1675
@@
 Connection ~ 2825 2750
 $Comp
-L CONN_01X02 P213
+L KarkSchematics-rescue:CONN_01X02 P213
 U 1 1 5AB7503B
 P 3525 1675
@@
 	3575 2250 3575 3050
 $Comp
-L CONN_01X02 P217
+L KarkSchematics-rescue:CONN_01X02 P217
 U 1 1 5AB7503C
 P 3975 1675
@@
 IGN_1_A
 $Comp
-L CONN_01X04 P206
+L KarkSchematics-rescue:CONN_01X04 P206
 U 1 1 5AB7503D
 P 2275 6850
@@
 TPS_1_GND
 $Comp
-L CONN_01X04 P220
+L KarkSchematics-rescue:CONN_01X04 P220
 U 1 1 5AB7503E
 P 4425 6850
@@
 IAC_2_2A
 $Comp
-L CONN_01X02 P212
+L KarkSchematics-rescue:CONN_01X02 P212
 U 1 1 5AB7503F
 P 3125 6850
@@
 $EndComp
 $Comp
-L CONN_01X02 P216
+L KarkSchematics-rescue:CONN_01X02 P216
 U 1 1 5AB75040
 P 3725 6850
