File: Kark/Schematics/EFI_latch.sch (KiCad schematic (older format))
At the start: 9 parts

Commit message: changes made last year
Connections:
- net EFI_En: now also U?.10, U?.11; no longer U?.13, U?.9
- new net: U?.13, U?.9
Changed lines of the file:
@@
 $Descr USLetter 11000 8500
 encoding utf-8
-Sheet 6 5
+Sheet 5 5
 Title "Kark - Gasoline Prototype"
 Date "2019-05-17"
@@
 Wire Wire Line
 	7625 3025 7625 3375
-Text HLabel 8025 2550 2    60   Output ~ 0
+Text HLabel 7975 3375 2    60   Output ~ 0
 EFI_En
-Wire Wire Line
-	8025 2550 7625 2550
-Connection ~ 7625 2550
 $Comp
 L 74xx:7402 U?
@@
 Text Notes 4550 1375 0    118  ~ 0
 EFI Latch System
+Wire Wire Line
+	7975 3375 7625 3375
+Connection ~ 7625 3375
 $EndSCHEMATC
