File: Sting/editsByMe/Arduino.sch (KiCad schematic (older format))
At the start: 6 parts

Commit message: Adding Madeline's files
Parts:
- P?: value Arduino -> Can
Connections:
- net at U?.25 (GND): now also P?.2 (P2), P?.4 (P4), U?.2 (GND), U?.4 (GND), U?.4 (GND), U?.5 (GND)
- net Throttle_5v renamed CANH
- net Throttle_in renamed CANL
Other:
- note removed: "DELETE THIS!"
- note removed: "NEED TO CHANGE ALL OF THIS!\nNOT USING ARDUINOS!"
- note removed: "PUT CAN THING HERE ---- NEED TO FIGURE OUT HOW TO DO IT!"
Changed lines of the file:
@@
 $Descr USLetter 11000 8500
 encoding utf-8
-Sheet 5 14
+Sheet 5 12
 Title "Arduino Breakout"
 Date "2017-01-04"
@@
 Servo_GND
 Text HLabel 3400 2825 0    60   Input ~ 0
-Throttle_in
+CANL
 Text HLabel 3400 2725 0    60   Output ~ 0
-Throttle_5v
+CANH
 Text HLabel 3400 2925 0    60   Input ~ 0
 GND
@@
 P 3650 2775
 F 0 "P?" H 3650 3025 50  0001 C CNN
-F 1 "Arduino" H 3725 3050 50  0000 C CNN
+F 1 "Can" H 3725 3050 50  0000 C CNN
 F 2 "" H 3650 2775 50  0000 C CNN
 F 3 "" H 3650 2775 50  0000 C CNN
@@
 Wire Wire Line
 	4125 3250 4125 4700
-Text Notes 7000 3250 0    60   ~ 12
-NEED TO CHANGE ALL OF THIS!\nNOT USING ARDUINOS!
-Text Notes 2600 6000 0    60   ~ 12
-PUT CAN THING HERE ---- NEED TO FIGURE OUT HOW TO DO IT!
-Text Notes 4450 1650 0    60   ~ 0
-DELETE THIS!
 $EndSCHEMATC

Commit message: Added rescue files
Parts:
- P? (x2): symbol Wiring-Diagram-v2-rescue:CONN_01X03 -> Wiring-Diagram-v2-rescue:CONN_01X03-Wiring-Diagram-v2-rescue
- P? (x2): symbol Wiring-Diagram-v2-rescue:CONN_01X04 -> Wiring-Diagram-v2-rescue:CONN_01X04-Wiring-Diagram-v2-rescue
- U?: symbol Supermileage:Arduino -> Wiring-Diagram-v2-rescue:Arduino-Supermileage
- U?: symbol Supermileage:5v-DC_DC -> Wiring-Diagram-v2-rescue:5v-DC_DC-Supermileage
Connections:
- net at U?.25 (GND): now also P?.2 (P2), P?.4 (P4), U?.2 (GND), U?.4 (GND), U?.4 (GND), U?.5 (GND)
Changed lines of the file:
@@
 $EndDescr
 $Comp
-L Supermileage:Arduino U?
+L Wiring-Diagram-v2-rescue:Arduino-Supermileage U?
 U 1 1 589816B6
 P 5425 3650
@@
 GND
 $Comp
-L Wiring-Diagram-v2-rescue:CONN_01X03 P?
+L Wiring-Diagram-v2-rescue:CONN_01X03-Wiring-Diagram-v2-rescue P?
 U 1 1 58983E27
 P 3650 3250
@@
 $EndComp
 $Comp
-L Wiring-Diagram-v2-rescue:CONN_01X03 P?
+L Wiring-Diagram-v2-rescue:CONN_01X03-Wiring-Diagram-v2-rescue P?
 U 1 1 58983E2D
 P 3800 3250
@@
 Connection ~ 4350 2725
 $Comp
-L Wiring-Diagram-v2-rescue:CONN_01X04 P?
+L Wiring-Diagram-v2-rescue:CONN_01X04-Wiring-Diagram-v2-rescue P?
 U 1 1 58986906
 P 3650 2775
@@
 $EndComp
 $Comp
-L Wiring-Diagram-v2-rescue:CONN_01X04 P?
+L Wiring-Diagram-v2-rescue:CONN_01X04-Wiring-Diagram-v2-rescue P?
 U 1 1 58986989
 P 3800 2775
@@
 	3400 2925 3450 2925
 $Comp
-L Supermileage:5v-DC_DC U?
+L Wiring-Diagram-v2-rescue:5v-DC_DC-Supermileage U?
 U 1 1 58987E67
 P 4925 2000
