File: Sting/editsByMe/Back_Of_Car.sch (KiCad schematic (older format))
At the start: 36 parts, among them M1 Starter Motor, SW11 Canopy, SW3 ExternalKill

Commit message: Adding Madeline's files
Connections:
- net at P?.6: no longer CR1.~ (R2)
- net at P?.8: now also U?.3 (12v)
- new net: CR1.~ (R2), P?.3
- new net: CR1.~ (R2), P?.6
- new net: P?.5, P?.6, P?.7
- now unconnected: P?.6
Other:
- note added: "Breakout Box"
- note removed: "Breakout Box\n"
- note removed: "Edited by Madeline Chairvolotti Date: 02-23-2019"
Changed lines of the file:
@@
 $Descr USLetter 8500 11000 portrait
 encoding utf-8
-Sheet 13 14
+Sheet 13 12
 Title "Sting - Gasoline Prototype"
 Date "2017-01-02"
@@
 	3925 5750 3925 5575
 Connection ~ 3925 5575
-Text HLabel 2575 3725 0    60   Input ~ 0
+Text Notes 3750 6300 0    50   ~ 0
+Breakout Box
+Text HLabel 2800 3650 0    50   Input ~ 0
 Relay_GND
-Wire Wire Line
-	3175 3725 3175 4125
-Wire Wire Line
-	2575 3725 3175 3725
-Wire Wire Line
-	3425 4225 3175 4125
-Text Notes 3750 6250 0    60   ~ 0
-Breakout Box\n
-Text Notes 3800 9400 0    60   ~ 0
-Edited by Madeline Chairvolotti Date: 02-23-2019
+Entry Wire Line
+	3350 3950 3450 4050
+Wire Wire Line
+	3350 3950 2800 3950
+Wire Wire Line
+	2800 3950 2800 3650
 $EndSCHEMATC

Commit message: Added rescue files
Parts:
- CR1: symbol Supermileage:Starter_Relay -> Wiring-Diagram-v2-rescue:Starter_Relay-Supermileage
- F?: symbol Wiring-Diagram-v2-rescue:FUSE -> Wiring-Diagram-v2-rescue:FUSE-Wiring-Diagram-v2-rescue
- L?: symbol Supermileage:Fuel_Injector -> Wiring-Diagram-v2-rescue:Fuel_Injector-Supermileage
- M1: symbol Supermileage:Motor -> Wiring-Diagram-v2-rescue:Motor-Supermileage
- P? (x10): symbol Wiring-Diagram-v2-rescue:CONN_01X04 -> Wiring-Diagram-v2-rescue:CONN_01X04-Wiring-Diagram-v2-rescue
- P?: symbol Supermileage:8_Terminal_Strip -> Wiring-Diagram-v2-rescue:8_Terminal_Strip-Supermileage
- P? (x8): symbol Wiring-Diagram-v2-rescue:CONN_01X02 -> Wiring-Diagram-v2-rescue:CONN_01X02-Wiring-Diagram-v2-rescue
- SW11: symbol Wiring-Diagram-v2-rescue:SW_Push -> Wiring-Diagram-v2-rescue:SW_Push-Wiring-Diagram-v2-rescue
- SW3: symbol Supermileage:SW_SPST -> Wiring-Diagram-v2-rescue:SW_SPST-Supermileage
- TH? (x2): symbol Wiring-Diagram-v2-rescue:THERMISTOR -> Wiring-Diagram-v2-rescue:THERMISTOR-Wiring-Diagram-v2-rescue
- TPS: symbol Wiring-Diagram-v2-rescue:POT -> Wiring-Diagram-v2-rescue:POT-Wiring-Diagram-v2-rescue
- U?: symbol Supermileage:RPM_Sensor -> Wiring-Diagram-v2-rescue:RPM_Sensor-Supermileage
- U?: symbol Supermileage:O2_Sensor -> Wiring-Diagram-v2-rescue:O2_Sensor-Supermileage
- U?: symbol Supermileage:Ignition -> Wiring-Diagram-v2-rescue:Ignition-Supermileage
- U?: symbol Supermileage:12v-DC_DC -> Wiring-Diagram-v2-rescue:12v-DC_DC-Supermileage
Connections:
- net at P?.6: no longer CR1.~ (R2)
- net at P?.8: now also U?.3 (12v)
- new net: CR1.~ (R2), P?.3
- new net: CR1.~ (R2), P?.6
- new net: P?.5, P?.6, P?.7
- now unconnected: P?.6
Changed lines of the file:
@@
 $EndDescr
 $Comp
-L Supermileage:Motor M1
+L Wiring-Diagram-v2-rescue:Motor-Supermileage M1
 U 1 1 57E6F264
 P 4925 4025
@@
 $EndComp
 $Comp
-L Supermileage:Starter_Relay CR1
+L Wiring-Diagram-v2-rescue:Starter_Relay-Supermileage CR1
 U 1 1 57E6F37B
 P 3975 3925
@@
 $EndComp
 $Comp
-L Supermileage:SW_SPST SW3
+L Wiring-Diagram-v2-rescue:SW_SPST-Supermileage SW3
 U 1 1 57FB6E88
 P 3575 4875
@@
 $EndSheet
 $Comp
-L Supermileage:RPM_Sensor U?
+L Wiring-Diagram-v2-rescue:RPM_Sensor-Supermileage U?
 U 1 1 58736630
 P 6050 7250
@@
 $EndComp
 $Comp
-L Supermileage:O2_Sensor U?
+L Wiring-Diagram-v2-rescue:O2_Sensor-Supermileage U?
 U 1 1 58736636
 P 6050 6800
@@
 EFI_GND
 $Comp
-L Wiring-Diagram-v2-rescue:CONN_01X04 P?
+L Wiring-Diagram-v2-rescue:CONN_01X04-Wiring-Diagram-v2-rescue P?
 U 1 1 587D9944
 P 3275 6700
@@
 $EndComp
 $Comp
-L Wiring-Diagram-v2-rescue:CONN_01X04 P?
+L Wiring-Diagram-v2-rescue:CONN_01X04-Wiring-Diagram-v2-rescue P?
 U 1 1 587D9B20
 P 3425 6700
@@
 $EndComp
 $Comp
-L Wiring-Diagram-v2-rescue:CONN_01X04 P?
+L Wiring-Diagram-v2-rescue:CONN_01X04-Wiring-Diagram-v2-rescue P?
 U 1 1 587DD173
 P 3425 7250
@@
 $EndComp
 $Comp
-L Wiring-Diagram-v2-rescue:CONN_01X04 P?
+L Wiring-Diagram-v2-rescue:CONN_01X04-Wiring-Diagram-v2-rescue P?
 U 1 1 587E05EC
 P 3275 7250
@@
 CAN_GND
 $Comp
-L Supermileage:8_Terminal_Strip P?
+L Wiring-Diagram-v2-rescue:8_Terminal_Strip-Supermileage P?
 U 1 1 587F01AE
 P 4725 2525
@@
 $EndComp
 $Comp
-L Wiring-Diagram-v2-rescue:FUSE F?
+L Wiring-Diagram-v2-rescue:FUSE-Wiring-Diagram-v2-rescue F?
 U 1 1 587FE842
 P 5875 3175
@@
 Lt_Blue
 $Comp
-L Wiring-Diagram-v2-rescue:POT TPS?
+L Wiring-Diagram-v2-rescue:POT-Wiring-Diagram-v2-rescue TPS?
 U 1 1 5893DA3D
 P 6000 7825
@@
 	5825 7750 5700 7750
 $Comp
-L Supermileage:Fuel_Injector L?
+L Wiring-Diagram-v2-rescue:Fuel_Injector-Supermileage L?
 U 1 1 5893FCDD
 P 6150 8250
@@
 	5850 8300 5700 8300
 $Comp
-L Supermileage:Ignition U?
+L Wiring-Diagram-v2-rescue:Ignition-Supermileage U?
 U 1 1 5894001C
 P 6150 8600
@@
 	5850 8550 5700 8550
 $Comp
-L Wiring-Diagram-v2-rescue:CONN_01X04 P?
+L Wiring-Diagram-v2-rescue:CONN_01X04-Wiring-Diagram-v2-rescue P?
 U 1 1 589435FC
 P 5500 6700
@@
 $EndComp
 $Comp
-L Wiring-Diagram-v2-rescue:CONN_01X04 P?
+L Wiring-Diagram-v2-rescue:CONN_01X04-Wiring-Diagram-v2-rescue P?
 U 1 1 5894426D
 P 5500 7250
@@
 $EndComp
 $Comp
-L Wiring-Diagram-v2-rescue:CONN_01X04 P?
+L Wiring-Diagram-v2-rescue:CONN_01X04-Wiring-Diagram-v2-rescue P?
 U 1 1 5894481D
 P 5500 7800
@@
 $EndComp
 $Comp
-L Wiring-Diagram-v2-rescue:CONN_01X02 P?
+L Wiring-Diagram-v2-rescue:CONN_01X02-Wiring-Diagram-v2-rescue P?
 U 1 1 58944FE1
 P 5500 8250
@@
 $EndComp
 $Comp
-L Wiring-Diagram-v2-rescue:CONN_01X02 P?
+L Wiring-Diagram-v2-rescue:CONN_01X02-Wiring-Diagram-v2-rescue P?
 U 1 1 5894539F
 P 5500 8600
@@
 $EndComp
 $Comp
-L Wiring-Diagram-v2-rescue:CONN_01X02 P?
+L Wiring-Diagram-v2-rescue:CONN_01X02-Wiring-Diagram-v2-rescue P?
 U 1 1 58945D6C
 P 5350 8600
@@
 $EndComp
 $Comp
-L Wiring-Diagram-v2-rescue:CONN_01X02 P?
+L Wiring-Diagram-v2-rescue:CONN_01X02-Wiring-Diagram-v2-rescue P?
 U 1 1 589461F6
 P 5350 8250
@@
 $EndComp
 $Comp
-L Wiring-Diagram-v2-rescue:CONN_01X04 P?
+L Wiring-Diagram-v2-rescue:CONN_01X04-Wiring-Diagram-v2-rescue P?
 U 1 1 589464BE
 P 5350 7800
@@
 $EndComp
 $Comp
-L Wiring-Diagram-v2-rescue:CONN_01X04 P?
+L Wiring-Diagram-v2-rescue:CONN_01X04-Wiring-Diagram-v2-rescue P?
 U 1 1 589466E5
 P 5350 7250
@@
 $EndComp
 $Comp
-L Wiring-Diagram-v2-rescue:CONN_01X04 P?
+L Wiring-Diagram-v2-rescue:CONN_01X04-Wiring-Diagram-v2-rescue P?
 U 1 1 5894690C
 P 5350 6700
@@
 	5075 8650 5150 8650
 $Comp
-L Wiring-Diagram-v2-rescue:THERMISTOR TH?
+L Wiring-Diagram-v2-rescue:THERMISTOR-Wiring-Diagram-v2-rescue TH?
 U 1 1 5894C2EE
 P 2575 8100
@@
 $EndComp
 $Comp
-L Wiring-Diagram-v2-rescue:THERMISTOR TH?
+L Wiring-Diagram-v2-rescue:THERMISTOR-Wiring-Diagram-v2-rescue TH?
 U 1 1 5894C50E
 P 2575 8650
@@
 	2225 8650 2325 8650
 $Comp
-L Wiring-Diagram-v2-rescue:CONN_01X02 P?
+L Wiring-Diagram-v2-rescue:CONN_01X02-Wiring-Diagram-v2-rescue P?
 U 1 1 5894F13E
 P 3275 8250
@@
 $EndComp
 $Comp
-L Wiring-Diagram-v2-rescue:CONN_01X02 P?
+L Wiring-Diagram-v2-rescue:CONN_01X02-Wiring-Diagram-v2-rescue P?
 U 1 1 5894FBB5
 P 3425 8250
@@
 	3625 8300 3725 8300
 $Comp
-L Wiring-Diagram-v2-rescue:CONN_01X02 P?
+L Wiring-Diagram-v2-rescue:CONN_01X02-Wiring-Diagram-v2-rescue P?
 U 1 1 5895025A
 P 3275 8600
@@
 $EndComp
 $Comp
-L Wiring-Diagram-v2-rescue:CONN_01X02 P?
+L Wiring-Diagram-v2-rescue:CONN_01X02-Wiring-Diagram-v2-rescue P?
 U 1 1 5895064C
 P 3425 8600
@@
 	3075 8650 2825 8650
 $Comp
-L Supermileage:12v-DC_DC U?
+L Wiring-Diagram-v2-rescue:12v-DC_DC-Supermileage U?
 U 1 1 589B1E06
 P 3425 2325
@@
 Canopy_GND
 $Comp
-L Wiring-Diagram-v2-rescue:SW_Push SW11
+L Wiring-Diagram-v2-rescue:SW_Push-Wiring-Diagram-v2-rescue SW11
 U 1 1 5AB67834
 P 3575 5575

Commit message: added things, namely edited EFI_BREAKOUT
Connections:
- net at P?.6: no longer CR1.~ (R2)
- net at P?.8: now also U?.3 (12v)
- new net: CR1.~ (R2), P?.3
- new net: CR1.~ (R2), P?.6
- new net: P?.5, P?.6, P?.7
- now unconnected: P?.6
Changed lines of the file:
@@
 $Descr USLetter 8500 11000 portrait
 encoding utf-8
-Sheet 13 12
+Sheet 12 13
 Title "Sting - Gasoline Prototype"
 Date "2017-01-02"
