File: Sting/editsByMe/EFI_Breakout.sch (KiCad schematic (older format))
At the start: 23 parts

Commit message: Adding Madeline's files
Other:
- note added: "ONLY ON STING!!!"
- note removed: "Edited by Madeline Chairvolotti Date: 02-23-2019"
Changed lines of the file:
@@
 $Descr USLetter 11000 8500
 encoding utf-8
-Sheet 14 14
+Sheet 14 12
 Title "EFI Breakout"
 Date "2017-01-04"
@@
 Text Label 6475 4450 0    60   ~ 0
 SEN_GND
+Text Notes 6925 4450 0    60   ~ 0
+ONLY ON STING!!!
+Text Notes 6925 2750 0    60   ~ 0
+ONLY ON STING
+Text Notes 6925 4250 0    60   ~ 0
+ONLY ON STING
 Text Label 6525 2450 0    60   ~ 0
 white
@@
 	6375 2450 7725 2450
 Wire Wire Line
-	2225 3150 4975 3150
-Wire Wire Line
 	2225 3150 2225 6300
 Wire Wire Line
@@
 Wire Wire Line
 	4975 3850 4375 3850
-Wire Wire Line
-	4975 3250 4275 3250
 Wire Wire Line
 	2825 3650 4975 3650
@@
 Wire Wire Line
 	2425 4850 2325 4850
+Entry Bus Bus
+	4650 3150 4750 3250
+Wire Wire Line
+	2225 3150 4975 3150
+Wire Wire Line
+	4275 3250 4975 3250
 Wire Bus Line
 	8975 1550 8975 5300
 Wire Bus Line
 	7825 2250 7825 5300
-Text Notes 6925 4450 0    60   ~ 0
-ONLY ON STING
-Text Notes 6925 4250 0    60   ~ 0
-ONLY ON STING
-Text Notes 6925 2750 0    60   ~ 0
-ONLY ON STING
-Text Notes 6350 6900 0    60   ~ 0
-Edited by Madeline Chairvolotti Date: 02-23-2019
 $EndSCHEMATC

Commit message: Added rescue files
Parts:
- J? (x2): symbol Wiring-Diagram-v2-rescue:DB25 -> Wiring-Diagram-v2-rescue:DB25-Wiring-Diagram-v2-rescue
- J?: symbol Wiring-Diagram-v2-rescue:DB37 -> Wiring-Diagram-v2-rescue:DB37-Wiring-Diagram-v2-rescue
- P? (x12): symbol Wiring-Diagram-v2-rescue:CONN_01X04 -> Wiring-Diagram-v2-rescue:CONN_01X04-Wiring-Diagram-v2-rescue
- P? (x8): symbol Wiring-Diagram-v2-rescue:CONN_01X02 -> Wiring-Diagram-v2-rescue:CONN_01X02-Wiring-Diagram-v2-rescue
Changed lines of the file:
@@
 $EndDescr
 $Comp
-L Wiring-Diagram-v2-rescue:DB25 J?
+L Wiring-Diagram-v2-rescue:DB25-Wiring-Diagram-v2-rescue J?
 U 1 1 586D10CA
 P 5425 3450
 AR Path="/57E22A72/586D10CA" Ref="J?"  Part="1"
 AR Path="/57E2AF30/5873550E/586D10CA" Ref="J?"  Part="1"
+AR Path="/586D10CA" Ref="J?"  Part="1"
 F 0 "J?" H 5475 4800 50  0001 C CNN
 F 1 "DB25" H 5375 2100 50  0000 C CNN
@@
 O2_3_Sen
 $Comp
-L Wiring-Diagram-v2-rescue:CONN_01X04 P?
+L Wiring-Diagram-v2-rescue:CONN_01X04-Wiring-Diagram-v2-rescue P?
 U 1 1 586D10CB
 P 2375 2050
 AR Path="/57E22A72/586D10CB" Ref="P?"  Part="1"
 AR Path="/57E2AF30/5873550E/586D10CB" Ref="P?"  Part="1"
+AR Path="/586D10CB" Ref="P?"  Part="1"
 F 0 "P?" V 2575 2050 50  0001 C CNN
 F 1 "O2 Sensor" V 2475 2050 50  0000 C CNN
@@
 $EndComp
 $Comp
-L Wiring-Diagram-v2-rescue:CONN_01X02 P?
+L Wiring-Diagram-v2-rescue:CONN_01X02-Wiring-Diagram-v2-rescue P?
 U 1 1 586D10CC
 P 3525 2050
@@
 $EndComp
 $Comp
-L Wiring-Diagram-v2-rescue:CONN_01X02 P?
+L Wiring-Diagram-v2-rescue:CONN_01X02-Wiring-Diagram-v2-rescue P?
 U 1 1 586D10CD
 P 3975 2050
@@
 $EndComp
 $Comp
-L Wiring-Diagram-v2-rescue:CONN_01X04 P?
+L Wiring-Diagram-v2-rescue:CONN_01X04-Wiring-Diagram-v2-rescue P?
 U 1 1 586D10CE
 P 2975 2050
 AR Path="/57E22A72/586D10CE" Ref="P?"  Part="1"
 AR Path="/57E2AF30/5873550E/586D10CE" Ref="P?"  Part="1"
+AR Path="/586D10CE" Ref="P?"  Part="1"
 F 0 "P?" V 3175 2050 50  0001 C CNN
 F 1 "RPM" V 3075 2050 50  0000 C CNN
@@
 $EndComp
 $Comp
-L Wiring-Diagram-v2-rescue:CONN_01X04 P?
+L Wiring-Diagram-v2-rescue:CONN_01X04-Wiring-Diagram-v2-rescue P?
 U 1 1 586D10CF
 P 1775 2050
 AR Path="/57E22A72/586D10CF" Ref="P?"  Part="1"
 AR Path="/57E2AF30/5873550E/586D10CF" Ref="P?"  Part="1"
+AR Path="/586D10CF" Ref="P?"  Part="1"
 F 0 "P?" V 1975 2050 50  0001 C CNN
 F 1 "Power" V 1875 2050 50  0000 C CNN
@@
 O2_1_GND
 $Comp
-L Wiring-Diagram-v2-rescue:DB25 J?
+L Wiring-Diagram-v2-rescue:DB25-Wiring-Diagram-v2-rescue J?
 U 1 1 586D10D0
 P 5925 3450
 AR Path="/57E22A72/586D10D0" Ref="J?"  Part="1"
 AR Path="/57E2AF30/5873550E/586D10D0" Ref="J?"  Part="1"
+AR Path="/586D10D0" Ref="J?"  Part="1"
 F 0 "J?" H 5975 4800 50  0001 C CNN
 F 1 "DB25" H 5875 2100 50  0000 C CNN
@@
 $EndComp
 $Comp
-L Wiring-Diagram-v2-rescue:DB37 J?
+L Wiring-Diagram-v2-rescue:DB37-Wiring-Diagram-v2-rescue J?
 U 1 1 586D10D1
 P 9925 3400
 AR Path="/57E22A72/586D10D1" Ref="J?"  Part="1"
 AR Path="/57E2AF30/5873550E/586D10D1" Ref="J?"  Part="1"
+AR Path="/586D10D1" Ref="J?"  Part="1"
 F 0 "J?" H 10025 5300 50  0001 C CNN
 F 1 "Megasquirt" H 9875 1450 50  0000 C CNN
@@
 CLT_2_B
 $Comp
-L Wiring-Diagram-v2-rescue:CONN_01X04 P?
+L Wiring-Diagram-v2-rescue:CONN_01X04-Wiring-Diagram-v2-rescue P?
 U 1 1 586D10D2
 P 2275 6500
 AR Path="/57E22A72/586D10D2" Ref="P?"  Part="1"
 AR Path="/57E2AF30/5873550E/586D10D2" Ref="P?"  Part="1"
+AR Path="/586D10D2" Ref="P?"  Part="1"
 F 0 "P?" V 2475 6500 50  0001 C CNN
 F 1 "Throttle Position Sensor" V 2375 6500 50  0000 C CNN
@@
 $EndComp
 $Comp
-L Wiring-Diagram-v2-rescue:CONN_01X04 P?
+L Wiring-Diagram-v2-rescue:CONN_01X04-Wiring-Diagram-v2-rescue P?
 U 1 1 586D10D3
 P 4425 6500
 AR Path="/57E22A72/586D10D3" Ref="P?"  Part="1"
 AR Path="/57E2AF30/5873550E/586D10D3" Ref="P?"  Part="1"
+AR Path="/586D10D3" Ref="P?"  Part="1"
 F 0 "P?" V 4625 6500 50  0001 C CNN
 F 1 "Stepper IAC" V 4525 6500 50  0000 C CNN
@@
 IAC_4_2B
 $Comp
-L Wiring-Diagram-v2-rescue:CONN_01X02 P?
+L Wiring-Diagram-v2-rescue:CONN_01X02-Wiring-Diagram-v2-rescue P?
 U 1 1 586D10D4
 P 3125 6500
@@
 $EndComp
 $Comp
-L Wiring-Diagram-v2-rescue:CONN_01X02 P?
+L Wiring-Diagram-v2-rescue:CONN_01X02-Wiring-Diagram-v2-rescue P?
 U 1 1 586D10D5
 P 3725 6500
@@
 	8975 4500 9075 4600
 $Comp
-L Wiring-Diagram-v2-rescue:CONN_01X04 P?
+L Wiring-Diagram-v2-rescue:CONN_01X04-Wiring-Diagram-v2-rescue P?
 U 1 1 586D10D6
 P 1125 2050
 AR Path="/57E22A72/586D10D6" Ref="P?"  Part="1"
 AR Path="/57E2AF30/5873550E/586D10D6" Ref="P?"  Part="1"
+AR Path="/586D10D6" Ref="P?"  Part="1"
 F 0 "P?" V 1325 2050 50  0001 C CNN
 F 1 "CAN" V 1225 2050 50  0000 C CNN
@@
 CAN_4_PWR
 $Comp
-L Wiring-Diagram-v2-rescue:CONN_01X04 P?
+L Wiring-Diagram-v2-rescue:CONN_01X04-Wiring-Diagram-v2-rescue P?
 U 1 1 586D346A
 P 1125 1750
 AR Path="/57E22A72/586D346A" Ref="P?"  Part="1"
 AR Path="/57E2AF30/5873550E/586D346A" Ref="P?"  Part="1"
+AR Path="/586D346A" Ref="P?"  Part="1"
 F 0 "P?" V 1325 1750 50  0001 C CNN
 F 1 "CAN" V 1225 1750 50  0000 C CNN
@@
 $EndComp
 $Comp
-L Wiring-Diagram-v2-rescue:CONN_01X04 P?
+L Wiring-Diagram-v2-rescue:CONN_01X04-Wiring-Diagram-v2-rescue P?
 U 1 1 586D3DFD
 P 1775 1750
 AR Path="/57E22A72/586D3DFD" Ref="P?"  Part="1"
 AR Path="/57E2AF30/5873550E/586D3DFD" Ref="P?"  Part="1"
+AR Path="/586D3DFD" Ref="P?"  Part="1"
 F 0 "P?" V 1975 1750 50  0001 C CNN
 F 1 "Power" V 1875 1750 50  0000 C CNN
@@
 P_1_GND
 $Comp
-L Wiring-Diagram-v2-rescue:CONN_01X04 P?
+L Wiring-Diagram-v2-rescue:CONN_01X04-Wiring-Diagram-v2-rescue P?
 U 1 1 586D56B8
 P 2375 1750
 AR Path="/57E22A72/586D56B8" Ref="P?"  Part="1"
 AR Path="/57E2AF30/5873550E/586D56B8" Ref="P?"  Part="1"
+AR Path="/586D56B8" Ref="P?"  Part="1"
 F 0 "P?" V 2575 1750 50  0001 C CNN
 F 1 "O2 Sensor" V 2475 1750 50  0000 C CNN
@@
 	2325 2250 2325 2350
 $Comp
-L Wiring-Diagram-v2-rescue:CONN_01X04 P?
+L Wiring-Diagram-v2-rescue:CONN_01X04-Wiring-Diagram-v2-rescue P?
 U 1 1 586D6E55
 P 2975 1750
 AR Path="/57E22A72/586D6E55" Ref="P?"  Part="1"
 AR Path="/57E2AF30/5873550E/586D6E55" Ref="P?"  Part="1"
+AR Path="/586D6E55" Ref="P?"  Part="1"
 F 0 "P?" V 3175 1750 50  0001 C CNN
 F 1 "RPM" V 3075 1750 50  0000 C CNN
@@
 Connection ~ 2825 2750
 $Comp
-L Wiring-Diagram-v2-rescue:CONN_01X02 P?
+L Wiring-Diagram-v2-rescue:CONN_01X02-Wiring-Diagram-v2-rescue P?
 U 1 1 586D7A2D
 P 3525 1750
@@
 	3575 2250 3575 3050
 $Comp
-L Wiring-Diagram-v2-rescue:CONN_01X02 P?
+L Wiring-Diagram-v2-rescue:CONN_01X02-Wiring-Diagram-v2-rescue P?
 U 1 1 586D8B07
 P 3975 1750
@@
 IGN_1_A
 $Comp
-L Wiring-Diagram-v2-rescue:CONN_01X04 P?
+L Wiring-Diagram-v2-rescue:CONN_01X04-Wiring-Diagram-v2-rescue P?
 U 1 1 586D9544
 P 2275 6850
 AR Path="/57E22A72/586D9544" Ref="P?"  Part="1"
 AR Path="/57E2AF30/5873550E/586D9544" Ref="P?"  Part="1"
+AR Path="/586D9544" Ref="P?"  Part="1"
 F 0 "P?" V 2475 6850 50  0001 C CNN
 F 1 "Throttle Position Sensor" V 2375 6850 50  0000 C CNN
@@
 TPS_1_GND
 $Comp
-L Wiring-Diagram-v2-rescue:CONN_01X04 P?
+L Wiring-Diagram-v2-rescue:CONN_01X04-Wiring-Diagram-v2-rescue P?
 U 1 1 586DAD2B
 P 4425 6850
 AR Path="/57E22A72/586DAD2B" Ref="P?"  Part="1"
 AR Path="/57E2AF30/5873550E/586DAD2B" Ref="P?"  Part="1"
+AR Path="/586DAD2B" Ref="P?"  Part="1"
 F 0 "P?" V 4625 6850 50  0001 C CNN
 F 1 "Stepper IAC" V 4525 6850 50  0000 C CNN
@@
 IAC_2_2A
 $Comp
-L Wiring-Diagram-v2-rescue:CONN_01X02 P?
+L Wiring-Diagram-v2-rescue:CONN_01X02-Wiring-Diagram-v2-rescue P?
 U 1 1 586DB7C8
 P 3125 6850
@@
 $EndComp
 $Comp
-L Wiring-Diagram-v2-rescue:CONN_01X02 P?
+L Wiring-Diagram-v2-rescue:CONN_01X02-Wiring-Diagram-v2-rescue P?
 U 1 1 586DCC77
 P 3725 6850

Commit message: added things, namely edited EFI_BREAKOUT
Connections:
- net GND: now also J?.1, J?.13, J?.3, P?.1 (P1), P?.1 (P1), P?.1 (P1), P?.1 (P1), P?.2 (P2), P?.2 (P2)
- net 12v: now reaches J?.6, P?.4 (P4), P?.4 (P4)
- net 12v: now also P?.1 (P1), P?.1 (P1)
Changed lines of the file:
@@
 $Descr USLetter 11000 8500
 encoding utf-8
-Sheet 14 12
+Sheet 13 13
 Title "EFI Breakout"
 Date "2017-01-04"
@@
 	1825 3050 1825 2250
 Wire Wire Line
-	1625 2750 2825 2750
-Wire Wire Line
-	1625 2750 1625 2250
-Wire Wire Line
 	1725 2250 1725 2350
 Wire Wire Line
 	3025 3050 3025 2250
 Wire Wire Line
-	2825 2250 2825 2750
-Wire Wire Line
 	2925 2250 2925 4350
 Wire Wire Line
@@
 	3925 2250 3925 2650
 Wire Wire Line
-	4025 2250 4025 3050
-Wire Wire Line
 	6375 3450 7725 3450
 Wire Wire Line
@@
 Wire Wire Line
 	4975 3850 4375 3850
-Wire Wire Line
-	2825 3650 4975 3650
 Wire Wire Line
 	4975 4450 4925 4450
@@
 	2925 4350 4975 4350
 Connection ~ 3125 3050
-Connection ~ 3575 3050
-Connection ~ 4025 3050
 Connection ~ 3025 3050
 Wire Wire Line
@@
 Wire Wire Line
 	3125 2250 3125 3050
-Connection ~ 2825 2750
 $Comp
 L Wiring-Diagram-v2-rescue:CONN_01X02-Wiring-Diagram-v2-rescue P?
@@
 Wire Wire Line
 	3475 3950 4975 3950
-Wire Wire Line
-	3575 2250 3575 3050
 $Comp
 L Wiring-Diagram-v2-rescue:CONN_01X02-Wiring-Diagram-v2-rescue P?
@@
 	1925 3050 2525 3050
 Wire Wire Line
-	3125 3050 3575 3050
-Wire Wire Line
-	3575 3050 4025 3050
-Wire Wire Line
-	4025 3050 4825 3050
-Wire Wire Line
 	3025 3050 3125 3050
 Wire Wire Line
@@
 	4825 3050 4825 4250
 Wire Wire Line
-	2825 2750 2825 3650
-Wire Wire Line
 	2425 4850 2325 4850
-Entry Bus Bus
-	4650 3150 4750 3250
 Wire Wire Line
 	2225 3150 4975 3150
 Wire Wire Line
 	4275 3250 4975 3250
+Wire Wire Line
+	3125 3050 4825 3050
+Text Label 1625 2775 1    60   ~ 0
+12v
+Text Label 2825 3500 1    60   ~ 0
+12v
+Text Label 3575 3500 1    60   ~ 0
+12v
+Text Label 2000 3050 0    60   ~ 0
+GND
+Text Label 4075 3050 0    60   ~ 0
+GND
+Text Label 4825 3500 1    60   ~ 0
+GND
+Wire Wire Line
+	1625 3650 2825 3650
+Text Label 1700 3650 0    60   ~ 0
+12v
+Wire Wire Line
+	1625 2250 1625 3650
+Wire Wire Line
+	2825 2250 2825 3650
+Connection ~ 2825 3650
+Wire Wire Line
+	2825 3650 3575 3650
+Wire Wire Line
+	3575 2250 3575 3650
+Connection ~ 3575 3650
+Wire Wire Line
+	3575 3650 4025 3650
+Wire Wire Line
+	4025 2250 4025 3650
 Wire Bus Line
 	8975 1550 8975 5300
 Wire Bus Line
 	7825 2250 7825 5300
+Connection ~ 4025 3650
+Wire Wire Line
+	4025 3650 4975 3650
+Text Label 4025 3500 1    60   ~ 0
+12v
+Text Label 2825 2775 1    60   ~ 0
+12v
+Text Label 3575 2775 1    60   ~ 0
+12v
 $EndSCHEMATC
