File: Sting/editsByMe/Relay_Box.sch (KiCad schematic (older format))
At the start: 22 parts, among them SW1 Master Power, SW10 SW_Push, SW12 Computer, SW2 Key, SW9 O2

Commit message: Adding Madeline's files
Connections:
- net Brown-Starter_PWR is gone; now on net Brown: R1.9 (C)
- net Orange-Horm is gone; now on net Brown: P?.8 (P8)
- net P_Green is gone; now on net Lt_Blue: P?.1 (P1), P?.3 (P3), P?.6 (P6), SW9.1 (C)
- net Red-PWR_LED is gone; now on net Brown: P?.5 (P5)
- net White-E_Start_SW is gone; now on net Blue: P?.3 (P3)
- net Yellow-EFI_LED is gone; now on net Purple-EFI_LED: P?.7 (P7)
- net Green: now also P?.2 (P2)
- net Lt_Blue-Arm_Status: now reaches R3.9 (C)
- net Blue-Sw_Power: no longer names the net of P?.4 (P4)
- net C_11_Wake_To_Parker renamed C_11_Wake
- net C_5_Horn_To_Parker renamed C_5_Horn
- net C_6_E_Stop_To_Parker renamed C_6_E_Stop
- net C_7_E_Start_To_Parker renamed C_7_E_Start
- net C_8_To_Parker: no longer names the net of P?.8 (P8)
- net C_9_Power_To_Parker renamed C_9_Power
- net E_9_RELAY_GND renamed E_9_RELAY_START_GND
- net Grey-To_Parker: no longer names the net of P?.8 (P8)
Other:
- note removed: "* Not using the Parker."
- note removed: "Edited by Madeline Chairvolotti Date: 02-23-2019"
Changed lines of the file:
@@
 $Descr USLetter 11000 8500
 encoding utf-8
-Sheet 4 14
+Sheet 4 12
 Title "Sting - Gasoline Prototype"
 Date "2017-01-04"
@@
 U 1 1 57FAAED6
 P 2100 2100
-AR Path="/57E6D70C/57FAAED6" Ref="SW2"  Part="1"
-AR Path="/5C847568/57FAAED6" Ref="SW?"  Part="1"
 F 0 "SW2" H 2100 2250 60  0000 C CNN
 F 1 "Key" H 2100 2000 60  0000 C CNN
@@
 U 1 1 57FAAF38
 P 2100 3350
-AR Path="/57E6D70C/57FAAF38" Ref="SW12"  Part="1"
-AR Path="/5C847568/57FAAF38" Ref="SW?"  Part="1"
 F 0 "SW12" H 1900 3475 60  0000 C CNN
 F 1 "Computer" H 2100 3250 60  0000 C CNN
@@
 U 1 1 57FAAF6A
 P 2100 1700
-AR Path="/57E6D70C/57FAAF6A" Ref="SW1"  Part="1"
-AR Path="/5C847568/57FAAF6A" Ref="SW?"  Part="1"
 F 0 "SW1" H 2100 1850 60  0000 C CNN
 F 1 "Master Power" H 2100 1600 60  0000 C CNN
@@
 U 1 1 57FB6243
 P 1500 1700
-AR Path="/57E6D70C/57FB6243" Ref="CB1"  Part="1"
-AR Path="/5C847568/57FB6243" Ref="CB?"  Part="1"
 F 0 "CB1" H 1500 1875 60  0000 C CNN
 F 1 "15A" H 1500 1625 60  0000 C CNN
@@
 U 1 1 57FB631C
 P 1500 2100
-AR Path="/57E6D70C/57FB631C" Ref="CB2"  Part="1"
-AR Path="/5C847568/57FB631C" Ref="CB?"  Part="1"
 F 0 "CB2" H 1500 2275 60  0000 C CNN
 F 1 "5A" H 1500 2025 60  0000 C CNN
@@
 U 1 1 57FB6351
 P 1500 2550
-AR Path="/57E6D70C/57FB6351" Ref="CB3"  Part="1"
-AR Path="/5C847568/57FB6351" Ref="CB?"  Part="1"
 F 0 "CB3" H 1500 2725 60  0000 C CNN
 F 1 "5A" H 1500 2475 60  0000 C CNN
@@
 U 1 1 57FB6389
 P 1500 4200
-AR Path="/57E6D70C/57FB6389" Ref="CB5"  Part="1"
-AR Path="/5C847568/57FB6389" Ref="CB?"  Part="1"
 F 0 "CB5" H 1500 4400 60  0000 C CNN
 F 1 "5A" H 1500 4125 60  0000 C CNN
@@
 U 1 1 58025EF3
 P 8575 3500
-AR Path="/57E6D70C/58025EF3" Ref="P?"  Part="1"
-AR Path="/5C847568/58025EF3" Ref="P?"  Part="1"
 F 0 "P?" H 8575 4150 50  0001 C CNN
 F 1 "Steering Wheel" V 8675 3500 50  0000 C CNN
@@
 U 1 1 58025FD5
 P 8550 2100
-AR Path="/57E6D70C/58025FD5" Ref="P?"  Part="1"
-AR Path="/5C847568/58025FD5" Ref="P?"  Part="1"
 F 0 "P?" H 8550 2750 50  0001 C CNN
 F 1 "To Engine" V 8650 2100 50  0000 C CNN
@@
 U 1 1 58026060
 P 8575 5300
-AR Path="/57E6D70C/58026060" Ref="P?"  Part="1"
-AR Path="/5C847568/58026060" Ref="P?"  Part="1"
 F 0 "P?" H 8575 5950 50  0001 C CNN
 F 1 "Computer" V 8675 5300 50  0000 C CNN
@@
 U 1 1 5804354D
 P 8775 5300
-AR Path="/57E6D70C/5804354D" Ref="P?"  Part="1"
-AR Path="/5C847568/5804354D" Ref="P?"  Part="1"
 F 0 "P?" H 8775 5950 50  0001 C CNN
 F 1 "Computer" V 8875 5300 50  0001 C CNN
@@
 U 1 1 58043E9C
 P 8775 3500
-AR Path="/57E6D70C/58043E9C" Ref="P?"  Part="1"
-AR Path="/5C847568/58043E9C" Ref="P?"  Part="1"
 F 0 "P?" H 8775 4150 50  0001 C CNN
 F 1 "To_Steering_Wheel" V 8875 3500 50  0001 C CNN
@@
 U 1 1 5804442E
 P 8775 2100
-AR Path="/57E6D70C/5804442E" Ref="P?"  Part="1"
-AR Path="/5C847568/5804442E" Ref="P?"  Part="1"
 F 0 "P?" H 8775 2750 50  0001 C CNN
 F 1 "To_Engine" V 8875 2100 50  0001 C CNN
@@
 C_12_GND
 Text HLabel 9375 5750 2    60   Output ~ 0
-C_11_Wake_To_Parker
+C_11_Wake
 Text HLabel 9375 5650 2    60   Output ~ 0
 C_10_CAN_Power
 Text HLabel 9375 5550 2    60   Output ~ 0
-C_9_Power_To_Parker
+C_9_Power
 Text HLabel 9375 5350 2    60   Input ~ 0
-C_7_E_Start_To_Parker
+C_7_E_Start
 Text HLabel 9375 5250 2    60   Input ~ 0
-C_6_E_Stop_To_Parker
+C_6_E_Stop
 Text HLabel 9375 5150 2    60   Input ~ 0
-C_5_Horn_To_Parker
+C_5_Horn
 $Comp
 L Wiring-Diagram-v2-rescue:CONN_01X04 P?
 U 1 1 581DEDA2
 P 8575 4400
-AR Path="/57E6D70C/581DEDA2" Ref="P?"  Part="1"
-AR Path="/5C847568/581DEDA2" Ref="P?"  Part="1"
 F 0 "P?" H 8575 4650 50  0001 C CNN
 F 1 "Horn" V 8675 4400 50  0000 C CNN
@@
 U 1 1 581DEE44
 P 8775 4400
-AR Path="/57E6D70C/581DEE44" Ref="P?"  Part="1"
-AR Path="/5C847568/581DEE44" Ref="P?"  Part="1"
 F 0 "P?" H 8775 4650 50  0001 C CNN
 F 1 "HORN" V 8875 4400 50  0001 C CNN
@@
 Text Label 8350 2150 2    49   ~ 0
 Black
-Text Label 7675 3000 1    49   ~ 0
+Text Label 7675 2950 1    49   ~ 0
 Black
 Text Label 8375 2950 2    49   ~ 0
-Purple
+Lt_Blue
 Text Label 6625 2250 0    49   ~ 0
 Blue-Starter_Relay
+Text Label 8125 3650 0    49   ~ 0
+Brown
 Text Label 8075 4350 1    49   ~ 0
 Black
+Text Label 8125 4450 0    49   ~ 0
+Brown
 Text Label 8125 5150 0    49   ~ 0
 Brown
@@
 U 1 1 57FB63C4
 P 1500 3350
-AR Path="/57E6D70C/57FB63C4" Ref="CB4"  Part="1"
-AR Path="/5C847568/57FB63C4" Ref="CB?"  Part="1"
 F 0 "CB4" H 1500 3525 60  0000 C CNN
 F 1 "5A" H 1500 3275 60  0000 C CNN
@@
 U 1 1 58871F7E
 P 2100 2650
-AR Path="/57E6D70C/58871F7E" Ref="SW9"  Part="1"
-AR Path="/5C847568/58871F7E" Ref="SW?"  Part="1"
 F 0 "SW9" H 2100 2525 60  0000 C CNN
 F 1 "O2" H 2050 2775 60  0000 C CNN
@@
 U 1 1 5887AA0F
 P 3725 3950
-AR Path="/57E6D70C/5887AA0F" Ref="R2"  Part="1"
-AR Path="/5C847568/5887AA0F" Ref="R?"  Part="1"
 F 0 "R2" H 3725 3950 60  0000 C CNN
 F 1 "4PDT_Relay_b" H 3725 4000 60  0001 C CNN
@@
 U 1 1 5887E21B
 P 3875 4950
-AR Path="/57E6D70C/5887E21B" Ref="D?"  Part="1"
-AR Path="/5C847568/5887E21B" Ref="D?"  Part="1"
 F 0 "D?" H 3875 5050 50  0001 C CNN
 F 1 "D" H 3875 4850 50  0001 C CNN
@@
 Text Label 4725 5825 1    49   ~ 0
 Black
+Text Label 4925 5825 1    49   ~ 0
+Lt_Blue-Arm_Status_C
 Text Label 5125 5825 1    49   ~ 0
 Green-E_Stop_C
@@
 Text Label 3975 5825 1    49   ~ 0
 Blue-E_Start_C
+Text Label 4825 5825 1    49   ~ 0
+Lt_Blue-Arm_Status
 Entry Wire Line
 	3875 5825 3975 5925
@@
 Red-Main_PWR
 Text Label 6625 2950 0    49   ~ 0
-Grey-E_Stop
+Green-E_Stop
+Text Label 6625 3150 0    49   ~ 0
+Blue-E_Start_SW
 Text Label 6625 3350 0    49   ~ 0
-Red-PWR_LED
+Brown-PWR_LED
 Text Label 6625 3550 0    49   ~ 0
-Yellow-EFI_LED
+Purple-EFI_LED
 Text Label 6625 4050 0    49   ~ 0
 Black
@@
 Text Label 7775 4900 1    49   ~ 0
 Brown
-Text Label 6875 4450 2    49   ~ 0
+Text Label 7775 4350 1    49   ~ 0
 Brown
 Text Label 7875 4350 1    49   ~ 0
@@
 U 1 1 58BF4D51
 P 4875 3950
-AR Path="/57E6D70C/58BF4D51" Ref="R3"  Part="1"
-AR Path="/5C847568/58BF4D51" Ref="R?"  Part="1"
 F 0 "R3" H 4875 3950 60  0000 C CNN
 F 1 "SPDT_Relay" V 5165 3920 60  0001 C CNN
@@
 U 1 1 59D1EFC0
 P 5625 3950
-AR Path="/57E6D70C/59D1EFC0" Ref="R1"  Part="1"
-AR Path="/5C847568/59D1EFC0" Ref="R?"  Part="1"
 F 0 "R1" H 5625 3950 60  0000 C CNN
 F 1 "SPDT_Relay" V 5915 3920 60  0001 C CNN
@@
 	1    0    0    -1
 $EndComp
+Text Label 6625 3450 0    49   ~ 0
+Brown-Starter_PWR
 Text Label 5625 5825 1    49   ~ 0
 Brown-Starter_PWR
@@
 Blue-Starter_Relay
 Text Label 6625 3050 0    49   ~ 0
-White-E_Start_SW
+Blue-E_Start_SW
 Entry Wire Line
 	6375 3150 6475 3050
@@
 Entry Wire Line
 	5775 5825 5875 5925
+Text Label 7900 2950 1    49   ~ 0
+Lt_Blue
 Text Label 8000 2950 1    49   ~ 0
 P_Green
@@
 P_Green
 Entry Wire Line
-	6375 2900 6475 2800
+	6375 3550 6475 3450
+Wire Wire Line
+	8350 1650 7900 1650
+Wire Wire Line
+	7900 1650 7900 2950
+Wire Wire Line
+	7900 2950 8375 2950
 Wire Wire Line
 	8375 3450 8000 3450
@@
 	8375 5150 7775 5150
 Wire Wire Line
+	7775 3650 8375 3650
+Wire Wire Line
 	2400 3350 2400 5825
 Wire Wire Line
@@
 	8975 2250 9375 2250
 Wire Wire Line
+	7775 3650 7775 4450
+Wire Wire Line
 	7775 4450 8375 4450
 Wire Wire Line
@@
 	8350 2550 6475 2550
 Wire Wire Line
-	7400 3250 8375 3250
+	7400 3050 8375 3050
+Wire Wire Line
+	8375 3150 6475 3150
 Wire Wire Line
 	8375 3550 6475 3550
@@
 Wire Wire Line
 	5775 4600 5775 5825
+Wire Wire Line
+	7850 3450 6475 3450
+Wire Wire Line
+	7850 3350 7850 3450
+Wire Wire Line
+	8375 3350 7850 3350
 Wire Wire Line
 	8050 3300 8375 3350
@@
 U 1 1 5AB5E5F2
 P 2075 3750
-AR Path="/57E6D70C/5AB5E5F2" Ref="SW10"  Part="1"
-AR Path="/5C847568/5AB5E5F2" Ref="SW?"  Part="1"
 F 0 "SW10" H 1900 3900 60  0000 C CNN
 F 1 "SW_Push" H 2075 3650 60  0000 C CNN
@@
 	6475 2350 8350 2350
 Text HLabel 9375 2350 2    60   Output ~ 0
-E_9_RELAY_GND
+E_9_RELAY_START_GND
 Wire Wire Line
 	9375 2350 8975 2350
-Wire Wire Line
-	7800 2950 7800 2800
-Wire Wire Line
-	7800 2800 6500 2800
-Wire Wire Line
-	7800 2950 8375 2950
-Entry Wire Line
-	6375 1750 6475 1650
-Wire Wire Line
-	6500 1650 8350 1650
-Wire Wire Line
-	7400 3250 7400 3150
-Wire Wire Line
-	7400 3150 6475 3150
-Text Label 6600 3150 0    47   ~ 0
-Blue-Sw_Power
-Entry Wire Line
-	6375 3750 6475 3650
-Wire Wire Line
-	6475 3650 8375 3650
-Entry Wire Line
-	6375 4550 6475 4450
-Wire Wire Line
-	8375 4450 6475 4450
-Text Label 6600 3650 0    60   ~ 0
-Orange-Horm
 Entry Wire Line
 	6375 3250 6475 3150
-Entry Wire Line
-	6375 3150 6475 3050
-Text Notes 6300 6900 0    60   ~ 0
-Edited by Madeline Chairvolotti Date: 02-23-2019
-Text HLabel 9375 5450 2    60   Output ~ 0
-C_8_To_Parker
-Wire Wire Line
-	8975 5450 9375 5450
-Text Label 6625 5450 0    49   ~ 0
-Grey-To_Parker
-Wire Wire Line
-	8375 5450 6475 5450
-Entry Wire Line
-	6375 5550 6475 5450
-Entry Wire Line
-	6375 5450 6475 5350
 Wire Bus Line
 	1900 5925 6375 5925
 Wire Bus Line
 	6375 1500 6375 5925
-Text Notes 9050 6050 0    60   ~ 0
-* Not using the Parker.
 $EndSCHEMATC

Commit message: Added rescue files
Parts:
- CB1, CB2, CB3, CB4, CB5: symbol Supermileage:CB -> Wiring-Diagram-v2-rescue:CB-Supermileage
- P? (x6): symbol Wiring-Diagram-v2-rescue:CONN_01X12 -> Wiring-Diagram-v2-rescue:CONN_01X12-Wiring-Diagram-v2-rescue
- P? (x2): symbol Wiring-Diagram-v2-rescue:CONN_01X04 -> Wiring-Diagram-v2-rescue:CONN_01X04-Wiring-Diagram-v2-rescue
- R1, R3: symbol Supermileage:SPDT_Relay -> Wiring-Diagram-v2-rescue:SPDT_Relay-Supermileage
- R2: symbol Supermileage:4PDT_Relay_b -> Wiring-Diagram-v2-rescue:4PDT_Relay_b-Supermileage
- SW1, SW12, SW2: symbol Supermileage:SW_SPST -> Wiring-Diagram-v2-rescue:SW_SPST-Supermileage
- SW10: symbol Wiring-Diagram-v2-rescue:SW_Push -> Wiring-Diagram-v2-rescue:SW_Push-Wiring-Diagram-v2-rescue
- SW9: symbol Supermileage:SW_SPDT -> Wiring-Diagram-v2-rescue:SW_SPDT-Supermileage
Changed lines of the file:
@@
 $EndDescr
 $Comp
-L Supermileage:SW_SPST SW2
+L Wiring-Diagram-v2-rescue:SW_SPST-Supermileage SW2
 U 1 1 57FAAED6
 P 2100 2100
@@
 $EndComp
 $Comp
-L Supermileage:SW_SPST SW12
+L Wiring-Diagram-v2-rescue:SW_SPST-Supermileage SW12
 U 1 1 57FAAF38
 P 2100 3350
@@
 $EndComp
 $Comp
-L Supermileage:SW_SPST SW1
+L Wiring-Diagram-v2-rescue:SW_SPST-Supermileage SW1
 U 1 1 57FAAF6A
 P 2100 1700
@@
 $EndComp
 $Comp
-L Supermileage:CB CB1
+L Wiring-Diagram-v2-rescue:CB-Supermileage CB1
 U 1 1 57FB6243
 P 1500 1700
@@
 $EndComp
 $Comp
-L Supermileage:CB CB2
+L Wiring-Diagram-v2-rescue:CB-Supermileage CB2
 U 1 1 57FB631C
 P 1500 2100
@@
 $EndComp
 $Comp
-L Supermileage:CB CB3
+L Wiring-Diagram-v2-rescue:CB-Supermileage CB3
 U 1 1 57FB6351
 P 1500 2550
@@
 $EndComp
 $Comp
-L Supermileage:CB CB5
+L Wiring-Diagram-v2-rescue:CB-Supermileage CB5
 U 1 1 57FB6389
 P 1500 4200
@@
 $EndComp
 $Comp
-L Wiring-Diagram-v2-rescue:CONN_01X12 P?
+L Wiring-Diagram-v2-rescue:CONN_01X12-Wiring-Diagram-v2-rescue P?
 U 1 1 58025EF3
 P 8575 3500
@@
 $EndComp
 $Comp
-L Wiring-Diagram-v2-rescue:CONN_01X12 P?
+L Wiring-Diagram-v2-rescue:CONN_01X12-Wiring-Diagram-v2-rescue P?
 U 1 1 58025FD5
 P 8550 2100
@@
 $EndComp
 $Comp
-L Wiring-Diagram-v2-rescue:CONN_01X12 P?
+L Wiring-Diagram-v2-rescue:CONN_01X12-Wiring-Diagram-v2-rescue P?
 U 1 1 58026060
 P 8575 5300
@@
 $EndComp
 $Comp
-L Wiring-Diagram-v2-rescue:CONN_01X12 P?
+L Wiring-Diagram-v2-rescue:CONN_01X12-Wiring-Diagram-v2-rescue P?
 U 1 1 5804354D
 P 8775 5300
@@
 $EndComp
 $Comp
-L Wiring-Diagram-v2-rescue:CONN_01X12 P?
+L Wiring-Diagram-v2-rescue:CONN_01X12-Wiring-Diagram-v2-rescue P?
 U 1 1 58043E9C
 P 8775 3500
@@
 $EndComp
 $Comp
-L Wiring-Diagram-v2-rescue:CONN_01X12 P?
+L Wiring-Diagram-v2-rescue:CONN_01X12-Wiring-Diagram-v2-rescue P?
 U 1 1 5804442E
 P 8775 2100
@@
 C_5_Horn
 $Comp
-L Wiring-Diagram-v2-rescue:CONN_01X04 P?
+L Wiring-Diagram-v2-rescue:CONN_01X04-Wiring-Diagram-v2-rescue P?
 U 1 1 581DEDA2
 P 8575 4400
@@
 $EndComp
 $Comp
-L Wiring-Diagram-v2-rescue:CONN_01X04 P?
+L Wiring-Diagram-v2-rescue:CONN_01X04-Wiring-Diagram-v2-rescue P?
 U 1 1 581DEE44
 P 8775 4400
@@
 S_W_11_THROTTLE
 $Comp
-L Supermileage:CB CB4
+L Wiring-Diagram-v2-rescue:CB-Supermileage CB4
 U 1 1 57FB63C4
 P 1500 3350
@@
 $EndComp
 $Comp
-L Supermileage:SW_SPDT SW9
+L Wiring-Diagram-v2-rescue:SW_SPDT-Supermileage SW9
 U 1 1 58871F7E
 P 2100 2650
@@
 $EndComp
 $Comp
-L Supermileage:4PDT_Relay_b R2
+L Wiring-Diagram-v2-rescue:4PDT_Relay_b-Supermileage R2
 U 1 1 5887AA0F
 P 3725 3950
@@
 Wires with a C sufix provide the same functionality as the non-C wire\nbut are connected to the computer.
 $Comp
-L Supermileage:SPDT_Relay R3
+L Wiring-Diagram-v2-rescue:SPDT_Relay-Supermileage R3
 U 1 1 58BF4D51
 P 4875 3950
@@
 $EndComp
 $Comp
-L Supermileage:SPDT_Relay R1
+L Wiring-Diagram-v2-rescue:SPDT_Relay-Supermileage R1
 U 1 1 59D1EFC0
 P 5625 3950
@@
 	7800 3350 6475 3350
 $Comp
-L Wiring-Diagram-v2-rescue:SW_Push SW10
+L Wiring-Diagram-v2-rescue:SW_Push-Wiring-Diagram-v2-rescue SW10
 U 1 1 5AB5E5F2
 P 2075 3750
