File: Sting/editsByMe/Wiring Diagram v2.sch (KiCad schematic (older format))
At the start: 31 parts

Commit message: Adding Madeline's files
Parts:
- removed P? (x2): CAN, symbol Wiring-Diagram-v2-rescue:CONN_01X04
- removed P? (x3): CONN_01X02, symbol Wiring-Diagram-v2-rescue:CONN_01X02
- P?: value Arduino -> Can
Connections:
- net Arduino/Servo_GND is gone; now on net Relay_GND: M?.2 (GND)
- net Arduino/Servo_out is gone; now on net Relay_GND: M?.3 (CTL)
- net Red is gone; now on net Relay_GND: P?.11 (P11), P?.5 (P5)
- net Blue: now also P?.2 (P2)
- net Grey: now also P?.8 (P8)
- net Lt_Blue: no longer P?.3 (P3)
- net Orange: now also P?.1 (P1)
- net Pink: no longer P?.3 (P3)
- net White: now also P?.3 (P3)
- net Arduino/Servo_5v renamed Relay_GND
- net Relay_GND: now also P?.12 (P12), P?.15 (P15), P?.2 (P2), P?.7 (P7), P?.7 (P7), P?.9 (P9)
- removed net Black: P?.1 (P1), P?.12 (P12), P?.15 (P15), P?.7 (P7), P?.9 (P9)
- net CM0711/J2_3_ARM_STATUS: no longer names the net of P?.3 (P3)
- net Relay Box (Box of Doom)/C_4_Arm_Status: no longer names the net of P?.4 (P4)
- removed net Yellow: P?.2 (P2), P?.2 (P2), P?.7 (P7)
Other:
- note added: "Date: 03-23-2019"
- note added: "Edited by: Madeline Chairvolotti"
- note removed: "Canopy Stuff - keep except Canopy_GND, change to Relay_Start_GND"
Changed lines of the file:
@@
 $Descr USLetter 8500 11000 portrait
 encoding utf-8
-Sheet 1 14
+Sheet 1 12
 Title "Sting - Gasoline Prototype"
 Date "2016-05-25"
@@
 F12 "J2_10_PITOT" I L 2000 7900 60
 F13 "J2_11_SYSTEM_V" I L 2000 8000 60
-F14 "J2_3_ARM_STATUS" I L 2000 7200 60
-F15 "J2_4_HIGH_P_EFI" I L 2000 7300 60
-F16 "J2_12_LOW_P_EFI" I L 2000 8100 60
-F17 "J2_6_ENGINE_START" O L 2000 7500 60
-F18 "J2_5_ENGINE_STOP" O L 2000 7400 60
-F19 "J1_6_SEN_5V" O L 2000 5450 60
-F20 "J1_11_SEN_GND" O L 2000 5950 60
-F21 "J1_3_CAN_H" B L 2000 5150 60
-F22 "J1_9_CAN_L" B L 2000 5750 60
+F14 "J2_4_HIGH_P_EFI" I L 2000 7300 60
+F15 "J2_12_LOW_P_EFI" I L 2000 8100 60
+F16 "J2_6_ENGINE_START" O L 2000 7500 60
+F17 "J2_5_ENGINE_STOP" O L 2000 7400 60
+F18 "J1_6_SEN_5V" O L 2000 5450 60
+F19 "J1_11_SEN_GND" O L 2000 5950 60
+F20 "J1_3_CAN_H" B L 2000 5150 60
+F21 "J1_9_CAN_L" B L 2000 5750 60
 $EndSheet
 $Comp
@@
 Entry Wire Line
 	800  6250 900  6350
-Entry Wire Line
-	800  7100 900  7200
 Entry Wire Line
 	800  7300 900  7400
@@
 F29 "C_1_5v" I L 3250 2700 60
 F30 "C_2_THROTTLE" I L 3250 2800 60
-F31 "C_4_Arm_Status" I L 3250 3000 60
-F32 "C_10_CAN_Power" I L 3250 3600 60
-F33 "E_6_CANOPY_SW" O R 4975 1600 60
-F34 "E_5_CANOPY_PWR" O R 4975 1500 60
-F35 "E_9_CANOPY_GND" O R 4975 1900 60
+F31 "C_10_CAN_Power" I L 3250 3600 60
+F32 "E_6_CANOPY_SW" O R 4975 1600 60
+F33 "E_5_CANOPY_PWR" O R 4975 1500 60
+F34 "E_9_CANOPY_GND" O R 4975 1900 60
 $EndSheet
 Entry Wire Line
@@
 Text Label 950  6050 0    60   ~ 0
 White
-Text Label 950  7200 0    60   ~ 0
-Lt_Blue
 Text Label 950  7400 0    60   ~ 0
 Green
@@
 	1900 6650 2000 6650
 Wire Wire Line
-	1900 7200 2000 7200
-Wire Wire Line
 	1900 7300 2000 7300
 Wire Wire Line
@@
 	3200 2800 3250 2800
 Wire Wire Line
-	3200 3000 3250 3000
-Wire Wire Line
 	3200 3100 3250 3100
 Wire Wire Line
@@
 Wire Wire Line
 	1350 6350 900  6350
-Wire Wire Line
-	1350 7200 900  7200
 Wire Wire Line
 	1350 7400 900  7400
@@
 P 1550 9300
 F 0 "P?" H 1550 9550 50  0001 C CNN
-F 1 "Arduino" H 1625 9025 50  0000 C CNN
+F 1 "Can" H 1625 9025 50  0000 C CNN
 F 2 "" H 1550 9300 50  0000 C CNN
 F 3 "" H 1550 9300 50  0000 C CNN
@@
 	800  5850 900  5950
 Text Label 950  9250 0    60   ~ 0
-Pink
+White
 Text Label 950  9350 0    60   ~ 0
-Yellow
+Blue
 Text Label 950  9450 0    60   ~ 0
-Black
+Orange
 Text Label 950  9150 0    60   ~ 0
 White
@@
 Text Label 5800 1100 0    60   ~ 0
 Lt_Blue
-$Sheet
-S 5350 7650 1250 1050
-U 588FE424
-F0 "Current Sensor" 60
-F1 "Current_Sensor.sch" 60
-F2 "Current1" O R 6600 8300 60
-F3 "Current2" O R 6600 8400 60
-F4 "Current3" O R 6600 8500 60
-F5 "CANH" B R 6600 7825 60
-F6 "CANL" B R 6600 7925 60
-F7 "In1_+" U L 5350 7775 60
-F8 "In1_-" U L 5350 7875 60
-F9 "In2_+" U L 5350 8125 60
-F10 "In2_-" U L 5350 8225 60
-F11 "In3_+" U L 5350 8475 60
-F12 "In3_-" U L 5350 8575 60
-F13 "A_Power" I R 6600 8200 60
-F14 "A_GND" I R 6600 8600 60
-F15 "CAN_Power" I R 6600 7725 60
-F16 "CAN_GND" I R 6600 8025 60
-$EndSheet
-$Comp
-L Wiring-Diagram-v2-rescue:CONN_01X04 P?
-U 1 1 5891E242
-P 6850 7875
-F 0 "P?" H 6850 8125 50  0001 C CNN
-F 1 "CAN" V 6950 7875 50  0001 C CNN
-F 2 "" H 6850 7875 50  0000 C CNN
-F 3 "" H 6850 7875 50  0000 C CNN
-	1    6850 7875
-	1    0    0    1
-$EndComp
-$Comp
-L Wiring-Diagram-v2-rescue:CONN_01X02 P?
-U 1 1 58921421
-P 5100 7825
-F 0 "P?" H 5100 7975 50  0001 C CNN
-F 1 "CONN_01X02" V 5200 7825 50  0001 C CNN
-F 2 "" H 5100 7825 50  0000 C CNN
-F 3 "" H 5100 7825 50  0000 C CNN
-	1    5100 7825
-	-1   0    0    1
-$EndComp
-$Comp
-L Wiring-Diagram-v2-rescue:CONN_01X02 P?
-U 1 1 58922A85
-P 5100 8175
-F 0 "P?" H 5100 8325 50  0001 C CNN
-F 1 "CONN_01X02" V 5200 8175 50  0001 C CNN
-F 2 "" H 5100 8175 50  0000 C CNN
-F 3 "" H 5100 8175 50  0000 C CNN
-	1    5100 8175
-	-1   0    0    1
-$EndComp
-$Comp
-L Wiring-Diagram-v2-rescue:CONN_01X02 P?
-U 1 1 58923A6F
-P 5100 8525
-F 0 "P?" H 5100 8675 50  0001 C CNN
-F 1 "CONN_01X02" V 5200 8525 50  0001 C CNN
-F 2 "" H 5100 8525 50  0000 C CNN
-F 3 "" H 5100 8525 50  0000 C CNN
-	1    5100 8525
-	-1   0    0    1
-$EndComp
-Wire Wire Line
-	5300 7775 5350 7775
-Wire Wire Line
-	5300 7875 5350 7875
-Wire Wire Line
-	5300 8125 5350 8125
-Wire Wire Line
-	5300 8225 5350 8225
-Wire Wire Line
-	5300 8475 5350 8475
-Wire Wire Line
-	5300 8575 5350 8575
-Wire Wire Line
-	6650 7725 6600 7725
-Wire Wire Line
-	6650 7825 6600 7825
-Wire Wire Line
-	6650 7925 6600 7925
-Wire Wire Line
-	6650 8025 6600 8025
-Wire Wire Line
-	7700 7725 7200 7725
-Wire Wire Line
-	7700 7825 7200 7825
-Wire Wire Line
-	7700 7925 7200 7925
-Wire Wire Line
-	7700 8025 7200 8025
-Entry Wire Line
-	7700 7725 7800 7625
-Entry Wire Line
-	7700 7825 7800 7725
-Entry Wire Line
-	7700 7925 7800 7825
-Entry Wire Line
-	7700 8025 7800 7925
-$Comp
-L Wiring-Diagram-v2-rescue:CONN_01X04 P?
-U 1 1 5892B628
-P 7000 7875
-F 0 "P?" H 7000 8125 50  0001 C CNN
-F 1 "CAN" H 7075 7600 50  0000 C CNN
-F 2 "" H 7000 7875 50  0000 C CNN
-F 3 "" H 7000 7875 50  0000 C CNN
-	1    7000 7875
-	-1   0    0    1
-$EndComp
-Text Label 7200 8025 0    60   ~ 0
-22g_gry
-Text Label 7200 7925 0    60   ~ 0
-CANL
-Text Label 7200 7825 0    60   ~ 0
-CANH
-Text Label 7200 7725 0    60   ~ 0
-White
 $Comp
 L Supermileage:Servo M?
@@
 	3200 9850 3300 9850
 Wire Wire Line
-	3300 9850 3300 9150
-Wire Wire Line
 	3300 9150 3200 9150
 Wire Wire Line
-	3200 9250 3350 9250
+	3200 9250 3300 9250
 Wire Wire Line
 	3350 9950 3200 9950
@@
 	3200 10050 3400 10050
 Wire Wire Line
-	3350 9250 3350 9950
-Wire Wire Line
-	3400 9350 3200 9350
+	3400 9350 3350 9350
 Wire Wire Line
 	3400 10050 3400 9350
@@
 F14 "Canopy_PWR" I L 6200 1500 60
 F15 "Canopy_SW" I L 6200 1600 60
-F16 "Canopy_GND" I L 6200 1900 60
 $EndSheet
 Text Label 2200 2000 0    60   ~ 0
@@
 Text Label 950  3200 0    60   ~ 0
 Lt_Blue
-Text Notes 4250 2600 0    60   ~ 0
-Canopy Stuff - keep except Canopy_GND, change to Relay_Start_GND
 Text Label 2100 2200 0    60   ~ 0
 Black_Orange
@@
 Text Label 5800 2100 0    60   ~ 0
 Red
+Text Notes 7500 2300 1    60   ~ 0
+22 guage grey ->
+Text Notes 3800 9500 0    60   ~ 0
+Edited by: Madeline Chairvolotti
+Text Notes 5300 9500 0    60   ~ 0
+Date: 03-23-2019
+Entry Wire Line
+	800  3300 900  3400
+Text Label 950  3400 0    60   ~ 0
+Grey
+Wire Wire Line
+	900  3400 2650 3400
+Text Label 3250 9150 0    60   ~ 0
+Red
+Text Label 3300 9250 0    60   ~ 0
+Black
+Wire Wire Line
+	3300 9250 3350 9250
+Text Label 3350 9350 0    60   ~ 0
+Yellow
+Wire Wire Line
+	3350 9350 3200 9350
+Wire Wire Line
+	3300 9150 3300 9850
+Wire Wire Line
+	3350 9250 3350 9950
+Text HLabel 6200 1900 2    60   Output ~ 0
+Relay_GND
 Wire Bus Line
 	900  4400 7800 4400
@@
 Wire Bus Line
 	800  2550 800  9450
-Text Notes 7500 2300 1    60   ~ 0
-22 guage grey ->
 $EndSCHEMATC

Commit message: Added rescue files
Parts:
- M?: symbol Supermileage:Servo -> Wiring-Diagram-v2-rescue:Servo-Supermileage
- P? (x4): symbol Wiring-Diagram-v2-rescue:CONN_01X18 -> Wiring-Diagram-v2-rescue:CONN_01X18-Wiring-Diagram-v2-rescue
- P? (x6): symbol Wiring-Diagram-v2-rescue:CONN_01X12 -> Wiring-Diagram-v2-rescue:CONN_01X12-Wiring-Diagram-v2-rescue
- P? (x14): symbol Wiring-Diagram-v2-rescue:CONN_01X04 -> Wiring-Diagram-v2-rescue:CONN_01X04-Wiring-Diagram-v2-rescue
- SP1: symbol Supermileage:Horn -> Wiring-Diagram-v2-rescue:Horn-Supermileage
Changed lines of the file:
@@
 $EndSheet
 $Comp
-L Wiring-Diagram-v2-rescue:CONN_01X18 P?
+L Wiring-Diagram-v2-rescue:CONN_01X18-Wiring-Diagram-v2-rescue P?
 U 1 1 586B46AB
 P 1700 5800
@@
 $EndComp
 $Comp
-L Wiring-Diagram-v2-rescue:CONN_01X18 P?
+L Wiring-Diagram-v2-rescue:CONN_01X18-Wiring-Diagram-v2-rescue P?
 U 1 1 586BFED3
 P 1700 7850
@@
 $EndComp
 $Comp
-L Wiring-Diagram-v2-rescue:CONN_01X18 P?
+L Wiring-Diagram-v2-rescue:CONN_01X18-Wiring-Diagram-v2-rescue P?
 U 1 1 58707A2D
 P 1550 5800
@@
 $EndComp
 $Comp
-L Wiring-Diagram-v2-rescue:CONN_01X18 P?
+L Wiring-Diagram-v2-rescue:CONN_01X18-Wiring-Diagram-v2-rescue P?
 U 1 1 58707FEE
 P 1550 7850
@@
 $EndComp
 $Comp
-L Wiring-Diagram-v2-rescue:CONN_01X12 P?
+L Wiring-Diagram-v2-rescue:CONN_01X12-Wiring-Diagram-v2-rescue P?
 U 1 1 58718B57
 P 3000 3250
@@
 $EndComp
 $Comp
-L Wiring-Diagram-v2-rescue:CONN_01X12 P?
+L Wiring-Diagram-v2-rescue:CONN_01X12-Wiring-Diagram-v2-rescue P?
 U 1 1 58721B64
 P 3000 1650
@@
 $EndComp
 $Comp
-L Wiring-Diagram-v2-rescue:CONN_01X12 P?
+L Wiring-Diagram-v2-rescue:CONN_01X12-Wiring-Diagram-v2-rescue P?
 U 1 1 58723F53
 P 2850 1650
@@
 $EndComp
 $Comp
-L Wiring-Diagram-v2-rescue:CONN_01X12 P?
+L Wiring-Diagram-v2-rescue:CONN_01X12-Wiring-Diagram-v2-rescue P?
 U 1 1 58739874
 P 5275 1650
@@
 $EndComp
 $Comp
-L Wiring-Diagram-v2-rescue:CONN_01X12 P?
+L Wiring-Diagram-v2-rescue:CONN_01X12-Wiring-Diagram-v2-rescue P?
 U 1 1 5873A376
 P 5425 1650
@@
 $EndComp
 $Comp
-L Wiring-Diagram-v2-rescue:CONN_01X04 P?
+L Wiring-Diagram-v2-rescue:CONN_01X04-Wiring-Diagram-v2-rescue P?
 U 1 1 587447E1
 P 5275 3650
@@
 $EndComp
 $Comp
-L Wiring-Diagram-v2-rescue:CONN_01X04 P?
+L Wiring-Diagram-v2-rescue:CONN_01X04-Wiring-Diagram-v2-rescue P?
 U 1 1 58745FFC
 P 5425 3650
@@
 $EndComp
 $Comp
-L Wiring-Diagram-v2-rescue:CONN_01X12 P?
+L Wiring-Diagram-v2-rescue:CONN_01X12-Wiring-Diagram-v2-rescue P?
 U 1 1 58752B64
 P 2850 3250
@@
 	1900 9450 2000 9450
 $Comp
-L Wiring-Diagram-v2-rescue:CONN_01X04 P?
+L Wiring-Diagram-v2-rescue:CONN_01X04-Wiring-Diagram-v2-rescue P?
 U 1 1 587A95C2
 P 1700 9300
@@
 $EndComp
 $Comp
-L Wiring-Diagram-v2-rescue:CONN_01X04 P?
+L Wiring-Diagram-v2-rescue:CONN_01X04-Wiring-Diagram-v2-rescue P?
 U 1 1 587A9C8F
 P 1550 9300
@@
 	7700 4950 7800 4850
 $Comp
-L Wiring-Diagram-v2-rescue:CONN_01X04 P?
+L Wiring-Diagram-v2-rescue:CONN_01X04-Wiring-Diagram-v2-rescue P?
 U 1 1 58841380
 P 4950 5100
@@
 $EndComp
 $Comp
-L Wiring-Diagram-v2-rescue:CONN_01X04 P?
+L Wiring-Diagram-v2-rescue:CONN_01X04-Wiring-Diagram-v2-rescue P?
 U 1 1 5884291A
 P 5100 5100
@@
 	5300 5250 5350 5250
 $Comp
-L Wiring-Diagram-v2-rescue:CONN_01X04 P?
+L Wiring-Diagram-v2-rescue:CONN_01X04-Wiring-Diagram-v2-rescue P?
 U 1 1 58849FE2
 P 4950 6450
@@
 $EndComp
 $Comp
-L Wiring-Diagram-v2-rescue:CONN_01X04 P?
+L Wiring-Diagram-v2-rescue:CONN_01X04-Wiring-Diagram-v2-rescue P?
 U 1 1 58849FE8
 P 5100 6450
@@
 	5300 6600 5350 6600
 $Comp
-L Wiring-Diagram-v2-rescue:CONN_01X04 P?
+L Wiring-Diagram-v2-rescue:CONN_01X04-Wiring-Diagram-v2-rescue P?
 U 1 1 5884A358
 P 4950 7050
@@
 $EndComp
 $Comp
-L Wiring-Diagram-v2-rescue:CONN_01X04 P?
+L Wiring-Diagram-v2-rescue:CONN_01X04-Wiring-Diagram-v2-rescue P?
 U 1 1 5884A35E
 P 5100 7050
@@
 	5300 7200 5350 7200
 $Comp
-L Wiring-Diagram-v2-rescue:CONN_01X04 P?
+L Wiring-Diagram-v2-rescue:CONN_01X04-Wiring-Diagram-v2-rescue P?
 U 1 1 5884C276
 P 6850 5100
@@
 $EndComp
 $Comp
-L Wiring-Diagram-v2-rescue:CONN_01X04 P?
+L Wiring-Diagram-v2-rescue:CONN_01X04-Wiring-Diagram-v2-rescue P?
 U 1 1 5884C27C
 P 7000 5100
@@
 	6600 5250 6650 5250
 $Comp
-L Wiring-Diagram-v2-rescue:CONN_01X04 P?
+L Wiring-Diagram-v2-rescue:CONN_01X04-Wiring-Diagram-v2-rescue P?
 U 1 1 5884EDF8
 P 6850 6450
@@
 $EndComp
 $Comp
-L Wiring-Diagram-v2-rescue:CONN_01X04 P?
+L Wiring-Diagram-v2-rescue:CONN_01X04-Wiring-Diagram-v2-rescue P?
 U 1 1 5884EDFE
 P 7000 6450
@@
 Lt_Blue
 $Comp
-L Supermileage:Servo M?
+L Wiring-Diagram-v2-rescue:Servo-Supermileage M?
 U 1 1 58993384
 P 2800 9950
@@
 	3400 10050 3400 9350
 $Comp
-L Supermileage:Horn SP1
+L Wiring-Diagram-v2-rescue:Horn-Supermileage SP1
 U 1 1 587EEE96
 P 5800 3750

Commit message: added things, namely edited EFI_BREAKOUT
Connections:
- net Arduino/GND renamed Throttle/GND
- net Arduino/Power renamed Throttle/Power
- net Arduino/Throttle_5v renamed Throttle/5v
- net Arduino/Throttle_in renamed Throttle/Throttle
Changed lines of the file:
@@
 $Descr USLetter 8500 11000 portrait
 encoding utf-8
-Sheet 1 12
+Sheet 1 13
 Title "Sting - Gasoline Prototype"
 Date "2016-05-25"
@@
 S 2000 9050 1200 525
 U 58788C84
-F0 "Arduino" 60
-F1 "Arduino.sch" 60
+F0 "Throttle" 60
+F1 "Throttle.sch" 60
 F2 "Power" I L 2000 9150 60
 F3 "GND" I L 2000 9450 60
@@
 F5 "Servo_out" O R 3200 9350 60
 F6 "Servo_GND" O R 3200 9250 60
-F7 "Throttle_in" I L 2000 9350 60
-F8 "Throttle_5v" O L 2000 9250 60
+F7 "Throttle" I L 2000 9350 60
+F8 "5v" O L 2000 9250 60
 $EndSheet
 Wire Wire Line
