File: Sting/wiring-diagrams/Arduino.sch (KiCad schematic (older format))
At the start: 6 parts

Commit message: fixed some stuff
Connections:
- net at U?.25 (GND): now also P?.2 (P2), P?.4 (P4), U?.2 (GND), U?.4 (GND), U?.4 (GND), U?.5 (GND)
Changed lines of the file:
@@
 LIBS:valves
 LIBS:Supermileage
-LIBS:Wiring Diagram v2-cache
+LIBS:EllicottDisplay
+LIBS:EllicottInterface
+LIBS:EllicottMicrocontrollers
+LIBS:EllicottMisc
+LIBS:EllicottPower
+LIBS:can_sensor-cache
+LIBS:pitot_tube-v1-cache
 EELAYER 25 0
 EELAYER END

Commit message: Made names consistant across pages
Connections:
- net at U?.25 (GND): now also P?.2 (P2), P?.4 (P4), U?.2 (GND), U?.4 (GND), U?.4 (GND), U?.5 (GND)
Changed lines of the file:
@@
 LIBS:EllicottMisc
 LIBS:EllicottPower
-LIBS:can_sensor-cache
-LIBS:pitot_tube-v1-cache
+LIBS:Wiring Diagram v2-cache
 EELAYER 25 0
 EELAYER END

Commit message: Moved where the relay to turn on the starter relay gets power from
Connections:
- net at U?.25 (GND): now also P?.2 (P2), P?.4 (P4), U?.2 (GND), U?.4 (GND), U?.4 (GND), U?.5 (GND)
Changed lines of the file:
@@
 EESchema Schematic File Version 2
+LIBS:Wiring Diagram v2-rescue
 LIBS:power
 LIBS:device

Commit message: Added Canopy Switches to Sting Documentation
Connections:
- net at U?.25 (GND): now also P?.2 (P2), P?.4 (P4), U?.2 (GND), U?.4 (GND), U?.4 (GND), U?.5 (GND)
Changed lines of the file:
@@
 LIBS:EllicottMisc
 LIBS:EllicottPower
+LIBS:relays_switches
 LIBS:Wiring Diagram v2-cache
 EELAYER 25 0

Commit message: Adding Madeline's files
Parts:
- P? (x2): symbol CONN_01X03 -> Wiring-Diagram-v2-rescue:CONN_01X03
- P? (x2): symbol CONN_01X04 -> Wiring-Diagram-v2-rescue:CONN_01X04
- U?: symbol Arduino -> Supermileage:Arduino
- U?: symbol 5v-DC_DC -> Supermileage:5v-DC_DC
Connections:
- net at U?.25 (GND): now also P?.2 (P2), P?.4 (P4), U?.2 (GND), U?.4 (GND), U?.4 (GND), U?.5 (GND)
Other:
- note added: "DELETE THIS!"
- note added: "Edited by Madeline Chairvolotti Date: 02-23-2019"
- note added: "NEED TO CHANGE ALL OF THIS!\nNOT USING ARDUINOS!"
- note added: "PUT CAN THING HERE ---- NEED TO FIGURE OUT HOW TO DO IT!"
Changed lines of the file:
@@
-EESchema Schematic File Version 2
-LIBS:Wiring Diagram v2-rescue
-LIBS:power
-LIBS:device
-LIBS:transistors
-LIBS:conn
-LIBS:linear
-LIBS:regul
-LIBS:74xx
-LIBS:cmos4000
-LIBS:adc-dac
-LIBS:memory
-LIBS:xilinx
-LIBS:microcontrollers
-LIBS:dsp
-LIBS:microchip
-LIBS:analog_switches
-LIBS:motorola
-LIBS:texas
-LIBS:intel
-LIBS:audio
-LIBS:interface
-LIBS:digital-audio
-LIBS:philips
-LIBS:display
-LIBS:cypress
-LIBS:siliconi
-LIBS:opto
-LIBS:atmel
-LIBS:contrib
-LIBS:valves
-LIBS:Supermileage
-LIBS:EllicottDisplay
-LIBS:EllicottInterface
-LIBS:EllicottMicrocontrollers
-LIBS:EllicottMisc
-LIBS:EllicottPower
-LIBS:relays_switches
+EESchema Schematic File Version 4
 LIBS:Wiring Diagram v2-cache
-EELAYER 25 0
+EELAYER 26 0
 EELAYER END
 $Descr USLetter 11000 8500
 encoding utf-8
-Sheet 7 14
+Sheet 5 14
 Title "Arduino Breakout"
 Date "2017-01-04"
@@
 $EndDescr
 $Comp
-L Arduino U?
+L Supermileage:Arduino U?
 U 1 1 589816B6
 P 5425 3650
@@
 GND
 $Comp
-L CONN_01X03 P?
+L Wiring-Diagram-v2-rescue:CONN_01X03 P?
 U 1 1 58983E27
 P 3650 3250
@@
 $EndComp
 $Comp
-L CONN_01X03 P?
+L Wiring-Diagram-v2-rescue:CONN_01X03 P?
 U 1 1 58983E2D
 P 3800 3250
@@
 	4350 3150 4000 3150
 Wire Wire Line
-	4350 2350 4350 3150
+	4350 2350 4350 2725
 Wire Wire Line
-	4000 2725 5325 2725
+	4000 2725 4350 2725
 Wire Wire Line
 	4000 2825 4575 2825
@@
 	4575 3150 4675 3150
 Wire Wire Line
-	4125 4700 5525 4700
+	4125 4700 5325 4700
 Wire Wire Line
 	5325 4700 5325 4500
@@
 Connection ~ 4350 2725
 $Comp
-L CONN_01X04 P?
+L Wiring-Diagram-v2-rescue:CONN_01X04 P?
 U 1 1 58986906
 P 3650 2775
@@
 $EndComp
 $Comp
-L CONN_01X04 P?
+L Wiring-Diagram-v2-rescue:CONN_01X04 P?
 U 1 1 58986989
 P 3800 2775
@@
 	4125 2925 4000 2925
 Wire Wire Line
-	4125 2100 4125 4700
+	4125 2100 4125 2250
 Wire Wire Line
 	3400 2725 3450 2725
@@
 	3400 2925 3450 2925
 $Comp
-L 5v-DC_DC U?
+L Supermileage:5v-DC_DC U?
 U 1 1 58987E67
 P 4925 2000
@@
 	4000 3250 4125 3250
 Connection ~ 4125 3250
+Wire Wire Line
+	5325 4700 5425 4700
+Wire Wire Line
+	5425 4700 5525 4700
+Wire Wire Line
+	4350 2725 4350 3150
+Wire Wire Line
+	4350 2725 5325 2725
+Wire Wire Line
+	4125 2925 4125 3250
+Wire Wire Line
+	4125 2250 4125 2925
+Wire Wire Line
+	4125 3250 4125 4700
+Text Notes 7000 3250 0    60   ~ 12
+NEED TO CHANGE ALL OF THIS!\nNOT USING ARDUINOS!
+Text Notes 2600 6000 0    60   ~ 12
+PUT CAN THING HERE ---- NEED TO FIGURE OUT HOW TO DO IT!
+Text Notes 4450 1650 0    60   ~ 0
+DELETE THIS!
+Text Notes 6350 7050 0    60   ~ 0
+Edited by Madeline Chairvolotti Date: 02-23-2019
 $EndSCHEMATC
