File: Sting/wiring-diagrams/Back_Of_Car.sch (KiCad schematic (older format))
At the start: 36 parts, among them M1 Starter Motor, SW11 Canopy, SW3 ExternalKill

Commit message: Adding Madeline's files
Parts:
- BT? (x2): symbol Battery -> Device:Battery
- CR1: symbol Starter_Relay -> Supermileage:Starter_Relay
- D?: symbol LED_ALT -> Device:LED_ALT
- F?: symbol FUSE -> Wiring-Diagram-v2-rescue:FUSE
- L1: symbol Electromagnetic_Actor -> Device:Electromagnetic_Actor
- L?: symbol Fuel_Injector -> Supermileage:Fuel_Injector
- M1: symbol Motor -> Supermileage:Motor
- P? (x10): symbol CONN_01X04 -> Wiring-Diagram-v2-rescue:CONN_01X04
- P?: symbol 8_Terminal_Strip -> Supermileage:8_Terminal_Strip
- P? (x8): symbol CONN_01X02 -> Wiring-Diagram-v2-rescue:CONN_01X02
- SW11: symbol SW_Push -> Wiring-Diagram-v2-rescue:SW_Push
- SW3: symbol SW_SPST -> Supermileage:SW_SPST
- TH? (x2): symbol THERMISTOR -> Wiring-Diagram-v2-rescue:THERMISTOR
- TPS: symbol POT -> Wiring-Diagram-v2-rescue:POT
- U?: symbol RPM_Sensor -> Supermileage:RPM_Sensor
- U?: symbol O2_Sensor -> Supermileage:O2_Sensor
- U?: symbol Ignition -> Supermileage:Ignition
- U?: symbol 12v-DC_DC -> Supermileage:12v-DC_DC
Connections:
- net at P?.6: no longer CR1.~ (R2)
- net at P?.8: now also U?.3 (12v)
- new net: CR1.~ (R2), P?.3
- new net: CR1.~ (R2), P?.6
- new net: P?.5, P?.6, P?.7
- now unconnected: P?.6
Other:
- note added: "Breakout Box\n"
- note added: "Edited by Madeline Chairvolotti Date: 02-23-2019"
Changed lines of the file:
@@
-EESchema Schematic File Version 2
-LIBS:Wiring Diagram v2-rescue
-LIBS:power
-LIBS:device
-LIBS:transistors
-LIBS:conn
-LIBS:linear
-LIBS:regul
-LIBS:74xx
-LIBS:cmos4000
-LIBS:adc-dac
-LIBS:memory
-LIBS:xilinx
-LIBS:microcontrollers
-LIBS:dsp
-LIBS:microchip
-LIBS:analog_switches
-LIBS:motorola
-LIBS:texas
-LIBS:intel
-LIBS:audio
-LIBS:interface
-LIBS:digital-audio
-LIBS:philips
-LIBS:display
-LIBS:cypress
-LIBS:siliconi
-LIBS:opto
-LIBS:atmel
-LIBS:contrib
-LIBS:valves
-LIBS:Supermileage
-LIBS:EllicottDisplay
-LIBS:EllicottInterface
-LIBS:EllicottMicrocontrollers
-LIBS:EllicottMisc
-LIBS:EllicottPower
-LIBS:relays_switches
+EESchema Schematic File Version 4
 LIBS:Wiring Diagram v2-cache
-EELAYER 25 0
+EELAYER 26 0
 EELAYER END
 $Descr USLetter 8500 11000 portrait
 encoding utf-8
-Sheet 3 14
+Sheet 13 14
 Title "Sting - Gasoline Prototype"
 Date "2017-01-02"
@@
 $EndDescr
 $Comp
-L Motor M1
+L Supermileage:Motor M1
 U 1 1 57E6F264
 P 4925 4025
@@
 $EndComp
 $Comp
-L Starter_Relay CR1
+L Supermileage:Starter_Relay CR1
 U 1 1 57E6F37B
 P 3975 3925
@@
 Engine_Start
 $Comp
-L Battery BT?
+L Device:Battery BT?
 U 1 1 57E6F190
 P 6275 3425
@@
 $EndComp
 $Comp
-L SW_SPST SW3
+L Supermileage:SW_SPST SW3
 U 1 1 57FB6E88
 P 3575 4875
@@
 $EndSheet
 $Comp
-L RPM_Sensor U?
+L Supermileage:RPM_Sensor U?
 U 1 1 58736630
 P 6050 7250
@@
 $EndComp
 $Comp
-L O2_Sensor U?
+L Supermileage:O2_Sensor U?
 U 1 1 58736636
 P 6050 6800
@@
 EFI_GND
 $Comp
-L CONN_01X04 P?
+L Wiring-Diagram-v2-rescue:CONN_01X04 P?
 U 1 1 587D9944
 P 3275 6700
@@
 $EndComp
 $Comp
-L CONN_01X04 P?
+L Wiring-Diagram-v2-rescue:CONN_01X04 P?
 U 1 1 587D9B20
 P 3425 6700
@@
 $EndComp
 $Comp
-L CONN_01X04 P?
+L Wiring-Diagram-v2-rescue:CONN_01X04 P?
 U 1 1 587DD173
 P 3425 7250
@@
 $EndComp
 $Comp
-L CONN_01X04 P?
+L Wiring-Diagram-v2-rescue:CONN_01X04 P?
 U 1 1 587E05EC
 P 3275 7250
@@
 CAN_GND
 $Comp
-L 8_Terminal_Strip P?
+L Supermileage:8_Terminal_Strip P?
 U 1 1 587F01AE
 P 4725 2525
@@
 $EndComp
 $Comp
-L FUSE F?
+L Wiring-Diagram-v2-rescue:FUSE F?
 U 1 1 587FE842
 P 5875 3175
@@
 $EndComp
 $Comp
-L Battery BT?
+L Device:Battery BT?
 U 1 1 5880064A
 P 6675 3425
@@
 Lt_Blue
 $Comp
-L POT TPS
+L Wiring-Diagram-v2-rescue:POT TPS?
 U 1 1 5893DA3D
 P 6000 7825
-AR Path="/5893DA3D" Ref="TPS"  Part="1"
+AR Path="/5893DA3D" Ref="TPS?"  Part="1"
 AR Path="/57E2AF30/5893DA3D" Ref="TPS"  Part="1"
 F 0 "TPS" V 6125 7700 50  0000 C CNN
@@
 	5825 7750 5700 7750
 $Comp
-L Fuel_Injector L?
+L Supermileage:Fuel_Injector L?
 U 1 1 5893FCDD
 P 6150 8250
@@
 	5850 8300 5700 8300
 $Comp
-L Ignition U?
+L Supermileage:Ignition U?
 U 1 1 5894001C
 P 6150 8600
@@
 	5850 8550 5700 8550
 $Comp
-L CONN_01X04 P?
+L Wiring-Diagram-v2-rescue:CONN_01X04 P?
 U 1 1 589435FC
 P 5500 6700
@@
 $EndComp
 $Comp
-L CONN_01X04 P?
+L Wiring-Diagram-v2-rescue:CONN_01X04 P?
 U 1 1 5894426D
 P 5500 7250
@@
 $EndComp
 $Comp
-L CONN_01X04 P?
+L Wiring-Diagram-v2-rescue:CONN_01X04 P?
 U 1 1 5894481D
 P 5500 7800
@@
 $EndComp
 $Comp
-L CONN_01X02 P?
+L Wiring-Diagram-v2-rescue:CONN_01X02 P?
 U 1 1 58944FE1
 P 5500 8250
+AR Path="/58944FE1" Ref="P?"  Part="1"
+AR Path="/57E2AF30/58944FE1" Ref="P?"  Part="1"
 F 0 "P?" H 5500 8400 50  0001 C CNN
 F 1 "Injector" H 5575 8075 50  0000 C CNN
@@
 $EndComp
 $Comp
-L CONN_01X02 P?
+L Wiring-Diagram-v2-rescue:CONN_01X02 P?
 U 1 1 5894539F
 P 5500 8600
+AR Path="/5894539F" Ref="P?"  Part="1"
+AR Path="/57E2AF30/5894539F" Ref="P?"  Part="1"
 F 0 "P?" H 5500 8750 50  0001 C CNN
 F 1 "Ignition" H 5575 8450 50  0000 C CNN
@@
 $EndComp
 $Comp
-L CONN_01X02 P?
+L Wiring-Diagram-v2-rescue:CONN_01X02 P?
 U 1 1 58945D6C
 P 5350 8600
+AR Path="/58945D6C" Ref="P?"  Part="1"
+AR Path="/57E2AF30/58945D6C" Ref="P?"  Part="1"
 F 0 "P?" H 5350 8750 50  0001 C CNN
 F 1 "Ignition" V 5450 8600 50  0001 C CNN
@@
 $EndComp
 $Comp
-L CONN_01X02 P?
+L Wiring-Diagram-v2-rescue:CONN_01X02 P?
 U 1 1 589461F6
 P 5350 8250
+AR Path="/589461F6" Ref="P?"  Part="1"
+AR Path="/57E2AF30/589461F6" Ref="P?"  Part="1"
 F 0 "P?" H 5350 8400 50  0001 C CNN
 F 1 "Injector" V 5450 8250 50  0001 C CNN
@@
 $EndComp
 $Comp
-L CONN_01X04 P?
+L Wiring-Diagram-v2-rescue:CONN_01X04 P?
 U 1 1 589464BE
 P 5350 7800
@@
 $EndComp
 $Comp
-L CONN_01X04 P?
+L Wiring-Diagram-v2-rescue:CONN_01X04 P?
 U 1 1 589466E5
 P 5350 7250
@@
 $EndComp
 $Comp
-L CONN_01X04 P?
+L Wiring-Diagram-v2-rescue:CONN_01X04 P?
 U 1 1 5894690C
 P 5350 6700
@@
 	5075 8650 5150 8650
 $Comp
-L THERMISTOR TH?
+L Wiring-Diagram-v2-rescue:THERMISTOR TH?
 U 1 1 5894C2EE
 P 2575 8100
@@
 $EndComp
 $Comp
-L THERMISTOR TH?
+L Wiring-Diagram-v2-rescue:THERMISTOR TH?
 U 1 1 5894C50E
 P 2575 8650
@@
 	2225 8650 2325 8650
 $Comp
-L CONN_01X02 P?
+L Wiring-Diagram-v2-rescue:CONN_01X02 P?
 U 1 1 5894F13E
 P 3275 8250
+AR Path="/5894F13E" Ref="P?"  Part="1"
+AR Path="/57E2AF30/5894F13E" Ref="P?"  Part="1"
 F 0 "P?" H 3275 8400 50  0001 C CNN
 F 1 "Air Temp" H 3350 8075 50  0000 C CNN
@@
 $EndComp
 $Comp
-L CONN_01X02 P?
+L Wiring-Diagram-v2-rescue:CONN_01X02 P?
 U 1 1 5894FBB5
 P 3425 8250
+AR Path="/5894FBB5" Ref="P?"  Part="1"
+AR Path="/57E2AF30/5894FBB5" Ref="P?"  Part="1"
 F 0 "P?" H 3425 8400 50  0001 C CNN
 F 1 "Air Temp" V 3525 8250 50  0001 C CNN
@@
 	3625 8300 3725 8300
 $Comp
-L CONN_01X02 P?
+L Wiring-Diagram-v2-rescue:CONN_01X02 P?
 U 1 1 5895025A
 P 3275 8600
+AR Path="/5895025A" Ref="P?"  Part="1"
+AR Path="/57E2AF30/5895025A" Ref="P?"  Part="1"
 F 0 "P?" H 3275 8750 50  0001 C CNN
 F 1 "Coolent Temp" H 3350 8425 50  0000 C CNN
@@
 $EndComp
 $Comp
-L CONN_01X02 P?
+L Wiring-Diagram-v2-rescue:CONN_01X02 P?
 U 1 1 5895064C
 P 3425 8600
+AR Path="/5895064C" Ref="P?"  Part="1"
+AR Path="/57E2AF30/5895064C" Ref="P?"  Part="1"
 F 0 "P?" H 3425 8750 50  0001 C CNN
 F 1 "Coolent" V 3525 8600 50  0001 C CNN
@@
 	3075 8650 2825 8650
 $Comp
-L 12v-DC_DC U?
+L Supermileage:12v-DC_DC U?
 U 1 1 589B1E06
 P 3425 2325
@@
 	6225 7825 6150 7825
 $Comp
-L LED_ALT D?
+L Device:LED_ALT D?
 U 1 1 58BFCDF3
 P 4375 4375
@@
 Canopy_GND
 $Comp
-L SW_Push SW11
+L Wiring-Diagram-v2-rescue:SW_Push SW11
 U 1 1 5AB67834
 P 3575 5575
@@
 $EndComp
 $Comp
-L Electromagnetic_Actor L1
+L Device:Electromagnetic_Actor L1
 U 1 1 5AB67BBC
 P 4275 5575
@@
 	3925 5750 3925 5575
 Connection ~ 3925 5575
+Text HLabel 2575 3725 0    60   Input ~ 0
+Relay_GND
+Wire Wire Line
+	3175 3725 3175 4125
+Wire Wire Line
+	2575 3725 3175 3725
+Wire Wire Line
+	3425 4225 3175 4125
+Text Notes 3750 6250 0    60   ~ 0
+Breakout Box\n
+Text Notes 3800 9400 0    60   ~ 0
+Edited by Madeline Chairvolotti Date: 02-23-2019
 $EndSCHEMATC
