File: Sting/wiring-diagrams/Pressure.sch (KiCad schematic (older format))
At the start: 23 parts

Commit message: fixed some stuff
Other:
- note added: "5v->3.3v Attenuator Select"
- note added: "Comments:\n\nQ1 and Q2 are reverse polarity protection transistors. They are P-Channel\nMosfets, so they have a very small resistance when on. \nCare should be taken in their selection so that their V-GS threshold is\nunder 1v\n\nU2 is a 5v regulator for the 5v pressure transducer. The output of U3 \ngoes through a selectable attenuator for a full 5v output or a 3.3v output.\n\nThere are position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"
- note added: "Full schematics with reference numbers are in the \npressure_sensor folder in the supermileagehw git repo at \nhttps://github.com/HEEV/supermileageHW"
- note removed: "Attenuator Selector"
- note removed: "Comments:\n\nQ1 and Q2 are reverse polarity protection transistors. They are P-Channel\nMosfets, so they have a very small resistance when on. \nCare should be taken in their selection so that their V-GS threshold is\nunder 1v\n\nU2 is a 5v regulator for the 5v pressure transducer. The output of U3 \ngoes through a selectable attenuator for a full 5v output or a 3.3v output."
- note removed: "Full schematics with reference numbers are in the \npressure_sensor folder in the supermileagehw git repo at \nhttps://bitbucket.org/nebk/supermileagehw"
- moved on the sheet: C?

Commit message: Adding Madeline's files
Parts:
- C? (x8): symbol C -> Device:C
- P? (x2): symbol CONN_01X04 -> Wiring-Diagram-v2-rescue:CONN_01X04
- P?: symbol CONN_01X03 -> Wiring-Diagram-v2-rescue:CONN_01X03
- Q? (x2): symbol Q_PMOS_GSD -> Device:Q_PMOS_GSD
- R? (x2): symbol R -> Device:R
- U?: symbol HSCDRR004MD -> Supermileage:HSCDRR004MD
- U?: symbol NJM2870F0 -> EllicottPower:NJM2870F0
- U?: symbol ASDX100A24R -> Supermileage:ASDX100A24R
- U?: symbol G4V-MINI -> Supermileage:G4V-MINI
- W? (x4): symbol TEST_1P -> Wiring-Diagram-v2-rescue:TEST_1P
Changed lines of the file:
@@
-EESchema Schematic File Version 2
-LIBS:Wiring Diagram v2-rescue
-LIBS:power
-LIBS:device
-LIBS:transistors
-LIBS:conn
-LIBS:linear
-LIBS:regul
-LIBS:74xx
-LIBS:cmos4000
-LIBS:adc-dac
-LIBS:memory
-LIBS:xilinx
-LIBS:microcontrollers
-LIBS:dsp
-LIBS:microchip
-LIBS:analog_switches
-LIBS:motorola
-LIBS:texas
-LIBS:intel
-LIBS:audio
-LIBS:interface
-LIBS:digital-audio
-LIBS:philips
-LIBS:display
-LIBS:cypress
-LIBS:siliconi
-LIBS:opto
-LIBS:atmel
-LIBS:contrib
-LIBS:valves
-LIBS:Supermileage
-LIBS:EllicottDisplay
-LIBS:EllicottInterface
-LIBS:EllicottMicrocontrollers
-LIBS:EllicottMisc
-LIBS:EllicottPower
-LIBS:relays_switches
+EESchema Schematic File Version 4
 LIBS:Wiring Diagram v2-cache
-EELAYER 25 0
+EELAYER 26 0
 EELAYER END
 $Descr USLetter 11000 8500
 encoding utf-8
-Sheet 9 14
+Sheet 10 14
 Title "Pressure Transducer Board"
 Date "2016-10-20"
@@
 $EndDescr
 $Comp
-L HSCDRR004MD U?
+L Supermileage:HSCDRR004MD U?
 U 1 1 58275680
 P 7600 5650
@@
 $EndComp
 $Comp
-L CONN_01X04 P?
+L Wiring-Diagram-v2-rescue:CONN_01X04 P?
 U 1 1 58275681
 P 2750 4500
@@
 $EndComp
 $Comp
-L C C?
+L Device:C C?
 U 1 1 58275682
 P 8350 5650
@@
 $EndComp
 $Comp
-L C C?
+L Device:C C?
 U 1 1 58275683
 P 8650 5650
@@
 $EndComp
 $Comp
-L GND #PWR?
+L power:GND #PWR?
 U 1 1 58275684
 P 8500 5900
@@
 $EndComp
 $Comp
-L +3.3V #PWR?
+L power:+3.3V #PWR?
 U 1 1 58275685
 P 8500 5400
@@
 $EndComp
 $Comp
-L +3.3V #PWR?
+L power:+3.3V #PWR?
 U 1 1 58275686
 P 7050 5450
@@
 $EndComp
 $Comp
-L GND #PWR?
+L power:GND #PWR?
 U 1 1 58275687
 P 3100 4800
@@
 $EndComp
 $Comp
-L GND #PWR?
+L power:GND #PWR?
 U 1 1 58275688
 P 3750 5300
@@
 $EndComp
 $Comp
-L GND #PWR?
+L power:GND #PWR?
 U 1 1 58275689
 P 7150 5950
@@
 Out
 $Comp
-L TEST_1P W?
+L Wiring-Diagram-v2-rescue:TEST_1P W?
 U 1 1 5827568A
 P 4075 3200
@@
 $EndComp
 $Comp
-L TEST_1P W?
+L Wiring-Diagram-v2-rescue:TEST_1P W?
 U 1 1 5827568B
 P 4425 3200
@@
 $EndComp
 $Comp
-L TEST_1P W?
+L Wiring-Diagram-v2-rescue:TEST_1P W?
 U 1 1 5827568C
 P 4725 3200
@@
 $EndComp
 $Comp
-L TEST_1P W?
+L Wiring-Diagram-v2-rescue:TEST_1P W?
 U 1 1 5827568D
 P 5075 3200
@@
 $EndComp
 $Comp
-L GND #PWR?
+L power:GND #PWR?
 U 1 1 5827568E
 P 4600 4400
@@
 $EndComp
 $Comp
-L NJM2870F0 U?
+L EllicottPower:NJM2870F0 U?
 U 1 1 5827568F
 P 4600 3650
@@
 $EndComp
 $Comp
-L C C?
+L Device:C C?
 U 1 1 58275690
 P 4050 4050
@@
 $EndComp
 $Comp
-L C C?
+L Device:C C?
 U 1 1 58275691
 P 5200 4150
@@
 $EndComp
 $Comp
-L C C?
+L Device:C C?
 U 1 1 58275692
 P 5800 4150
@@
 $EndComp
 $Comp
-L C C?
+L Device:C C?
 U 1 1 58275693
 P 5500 4150
@@
 Molex DuraClik
 $Comp
-L CONN_01X03 P?
+L Wiring-Diagram-v2-rescue:CONN_01X03 P?
 U 1 1 58275694
 P 6650 2950
@@
 5v->3.3v Attenuator Select
 $Comp
-L +5V #PWR?
+L power:+5V #PWR?
 U 1 1 58275695
 P 5800 3600
@@
 $EndComp
 $Comp
-L +5V #PWR?
+L power:+5V #PWR?
 U 1 1 58275696
 P 7050 3100
@@
 $EndComp
 $Comp
-L GND #PWR?
+L power:GND #PWR?
 U 1 1 58275697
 P 7050 4000
@@
 Out
 $Comp
-L R R?
+L Device:R R?
 U 1 1 58275698
 P 6550 3350
@@
 $EndComp
 $Comp
-L R R?
+L Device:R R?
 U 1 1 58275699
 P 6550 3750
@@
 	8350 5800 8350 5850
 Wire Wire Line
-	8350 5850 8650 5850
+	8350 5850 8500 5850
 Wire Wire Line
 	8650 5850 8650 5800
@@
 	8350 5500 8350 5450
 Wire Wire Line
-	8350 5450 8650 5450
+	8350 5450 8500 5450
 Wire Wire Line
 	8650 5450 8650 5500
@@
 	3400 3850 3550 3850
 Wire Wire Line
-	4600 4300 4600 4400
-Wire Wire Line
-	3750 4350 5800 4350
-Wire Wire Line
-	3950 3850 4100 3850
+	4600 4300 4600 4350
+Wire Wire Line
+	3750 4350 4050 4350
+Wire Wire Line
+	3950 3850 4050 3850
 Wire Wire Line
 	4100 3650 4050 3650
 Wire Wire Line
-	4050 3650 4050 3900
+	4050 3650 4050 3850
 Connection ~ 4050 3850
 Wire Wire Line
@@
 Connection ~ 4600 4350
 Wire Wire Line
-	5100 3650 5800 3650
+	5100 3650 5500 3650
 Wire Wire Line
 	5500 3650 5500 4000
@@
 Connection ~ 5500 4350
 Wire Wire Line
-	5800 3600 5800 4000
+	5800 3600 5800 3650
 Connection ~ 5500 3650
 Connection ~ 5800 3650
@@
 	7200 3550 7050 3550
 Wire Wire Line
-	7050 3550 7050 4000
+	7050 3550 7050 3950
 Wire Wire Line
 	7200 3450 6650 3450
 Wire Wire Line
-	6650 3150 6650 4650
+	6650 3150 6650 3450
 Wire Wire Line
 	6750 3250 6950 3250
@@
 	6550 3150 6550 3200
 Wire Wire Line
-	6550 3500 6550 3600
+	6550 3500 6550 3550
 Wire Wire Line
 	7050 3950 6550 3950
@@
 Connection ~ 6550 3550
 $Comp
-L C C?
+L Device:C C?
 U 1 1 5827569A
 P 8300 3500
@@
 $EndComp
 $Comp
-L C C?
+L Device:C C?
 U 1 1 5827569B
 P 8650 3500
@@
 $EndComp
 $Comp
-L +5V #PWR?
+L power:+5V #PWR?
 U 1 1 5827569C
 P 8500 3250
@@
 $EndComp
 $Comp
-L GND #PWR?
+L power:GND #PWR?
 U 1 1 5827569D
 P 8500 3750
@@
 	8300 3650 8300 3700
 Wire Wire Line
-	8300 3700 8650 3700
+	8300 3700 8500 3700
 Wire Wire Line
 	8650 3700 8650 3650
@@
 	8300 3350 8300 3300
 Wire Wire Line
-	8300 3300 8650 3300
+	8300 3300 8500 3300
 Wire Wire Line
 	8650 3300 8650 3350
@@
 Connection ~ 8500 3300
 $Comp
-L Q_PMOS_GSD Q?
+L Device:Q_PMOS_GSD Q?
 U 1 1 5827569E
 P 3750 3950
@@
 	3400 4350 3400 3850
 $Comp
-L Q_PMOS_GSD Q?
+L Device:Q_PMOS_GSD Q?
 U 1 1 5827569F
 P 3750 5050
@@
 5V absolute pressure transducer
 $Comp
-L +3.3V #PWR?
+L power:+3.3V #PWR?
 U 1 1 582756A0
 P 4100 4950
@@
 	6750 3150 6750 3250
 $Comp
-L ASDX100A24R U?
+L Supermileage:ASDX100A24R U?
 U 1 1 582756A1
 P 7600 3500
@@
 $EndComp
 $Comp
-L G4V-MINI U?
+L Supermileage:G4V-MINI U?
 U 1 1 582756A2
 P 7700 4600
@@
 $EndComp
 $Comp
-L +5V #PWR?
+L power:+5V #PWR?
 U 1 1 582756A3
 P 7050 4400
@@
 Connection ~ 6650 3450
 $Comp
-L GND #PWR?
+L power:GND #PWR?
 U 1 1 582756A4
 P 7050 4800
@@
 5V differential pressure transducer
 $Comp
-L CONN_01X04 P?
+L Wiring-Diagram-v2-rescue:CONN_01X04 P?
 U 1 1 58276BE6
 P 2400 4500
@@
 Text Notes 625  2900 0    60   ~ 0
 Comments:\n\nQ1 and Q2 are reverse polarity protection transistors. They are P-Channel\nMosfets, so they have a very small resistance when on. \nCare should be taken in their selection so that their V-GS threshold is\nunder 1v\n\nU2 is a 5v regulator for the 5v pressure transducer. The output of U3 \ngoes through a selectable attenuator for a full 5v output or a 3.3v output.\n\nThere are positions for three pressure transducers on this board; \nhowever only one of them can be populated at a time. The top two\ntransducers are 5v and have a selectable attenuator for using with a\n3.3v microcontroller. The bottom transducer is 3.3v.\n\nThe connector is a Molex DuraClik Part numbers are as follows\nFemale Socket:\nDigiKey:  WM12262-ND\nMouser: 538-505151-0400\nPCB Header:\nDigiKey: WM7171CT-ND\nMouser: 538-502352-0400\nPins:\nDigiKey: WM12344CT-ND\nMouser: 538-505153-8000-CT
+Wire Wire Line
+	8500 5850 8650 5850
+Wire Wire Line
+	8500 5450 8650 5450
+Wire Wire Line
+	4050 3850 4100 3850
+Wire Wire Line
+	4050 3850 4050 3900
+Wire Wire Line
+	4050 4350 4600 4350
+Wire Wire Line
+	4600 4350 4600 4400
+Wire Wire Line
+	4600 4350 5200 4350
+Wire Wire Line
+	5200 4350 5500 4350
+Wire Wire Line
+	5500 4350 5800 4350
+Wire Wire Line
+	5500 3650 5800 3650
+Wire Wire Line
+	5800 3650 5800 4000
+Wire Wire Line
+	7050 3950 7050 4000
+Wire Wire Line
+	6550 3550 6550 3600
+Wire Wire Line
+	8500 3700 8650 3700
+Wire Wire Line
+	8500 3300 8650 3300
+Wire Wire Line
+	6650 3450 6650 4650
 $EndSCHEMATC
