File: Sting/wiring-diagrams/Steering_Wheel.sch (KiCad schematic (older format))
At the start: 14 parts, among them SW4 Driver Kill, SW5 Engine Start, SW6 Engine Stop, SW7 Horn, SW8 Horn

Commit message: fixed missing parts updated sensor boards
Changed lines of the file:
@@
 	3150 6575 3350 6575
 Wire Wire Line
-	3750 5525 4000 5525
+	3750 5525 4300 5525
 Wire Wire Line
 	4000 6075 3750 6075
@@
 	5850 4925 5850 5325
 Wire Wire Line
-	4000 5325 5850 5325
-Wire Wire Line
-	5850 5325 5950 5325
+	4000 5325 5950 5325
 Connection ~ 5850 5325
 Wire Wire Line
 	6350 4925 6450 4925
 Wire Wire Line
-	6450 4925 6450 5325
-Wire Wire Line
-	6450 5325 6450 7325
+	6450 4925 6450 7325
 Wire Wire Line
 	6450 5325 6350 5325
@@
 	5450 5525 5000 5525
 Wire Wire Line
-	4000 5525 4000 5525
+	4000 5525 4000 6925
 Wire Wire Line
-	4000 5525 4000 6075
-Wire Wire Line
-	4000 6075 4000 6575
-Wire Wire Line
-	4000 6575 4000 6925
-Wire Wire Line
-	4000 5525 4300 5525
-Wire Wire Line
-	4300 5075 4000 5075
-Wire Wire Line
-	4000 5075 3150 5075
+	3150 5075 4300 5075
 Wire Wire Line
 	4300 4775 3150 4775
@@
 	5450 7125 3150 7125
 Wire Wire Line
-	5450 3975 5450 4425
-Wire Wire Line
-	5450 4425 5450 4775
-Wire Wire Line
-	5450 4775 5450 5075
-Wire Wire Line
-	5450 5075 5450 5525
-Wire Wire Line
-	5450 5525 5450 7125
+	5450 3975 5450 7125
 Wire Wire Line
 	6450 7325 3150 7325

Commit message: Adding Madeline's files
Parts:
- D? (x4): symbol Led_Small -> Wiring-Diagram-v2-rescue:Led_Small
- R? (x4): symbol R -> Device:R
- SW4: symbol SW_SPST -> Supermileage:SW_SPST
- SW5, SW6, SW7, SW8: symbol SW_NO -> Supermileage:SW_NO
- U?: symbol Throttle -> Supermileage:Throttle
Changed lines of the file:
@@
-EESchema Schematic File Version 2
-LIBS:Wiring Diagram v2-rescue
-LIBS:power
-LIBS:device
-LIBS:transistors
-LIBS:conn
-LIBS:linear
-LIBS:regul
-LIBS:74xx
-LIBS:cmos4000
-LIBS:adc-dac
-LIBS:memory
-LIBS:xilinx
-LIBS:microcontrollers
-LIBS:dsp
-LIBS:microchip
-LIBS:analog_switches
-LIBS:motorola
-LIBS:texas
-LIBS:intel
-LIBS:audio
-LIBS:interface
-LIBS:digital-audio
-LIBS:philips
-LIBS:display
-LIBS:cypress
-LIBS:siliconi
-LIBS:opto
-LIBS:atmel
-LIBS:contrib
-LIBS:valves
-LIBS:Supermileage
-LIBS:EllicottDisplay
-LIBS:EllicottInterface
-LIBS:EllicottMicrocontrollers
-LIBS:EllicottMisc
-LIBS:EllicottPower
-LIBS:relays_switches
+EESchema Schematic File Version 4
 LIBS:Wiring Diagram v2-cache
-EELAYER 25 0
+EELAYER 26 0
 EELAYER END
 $Descr USLetter 8500 11000 portrait
@@
 $EndDescr
 $Comp
-L SW_NO SW5
+L Supermileage:SW_NO SW5
 U 1 1 57E14402
 P 3550 6575
@@
 $EndComp
 $Comp
-L SW_NO SW7
+L Supermileage:SW_NO SW7
 U 1 1 57E14F53
 P 6150 4925
@@
 $EndComp
 $Comp
-L SW_NO SW6
+L Supermileage:SW_NO SW6
 U 1 1 57E1500F
 P 3550 6075
@@
 $EndComp
 $Comp
-L Throttle U?
+L Supermileage:Throttle U?
 U 1 1 57E1510C
 P 5800 4025
@@
 $EndComp
 $Comp
-L Led_Small D?
+L Wiring-Diagram-v2-rescue:Led_Small D?
 U 1 1 57E152BF
 P 4400 5075
@@
 $EndComp
 $Comp
-L Led_Small D?
+L Wiring-Diagram-v2-rescue:Led_Small D?
 U 1 1 57E153DC
 P 4400 4775
@@
 $EndComp
 $Comp
-L Led_Small D?
+L Wiring-Diagram-v2-rescue:Led_Small D?
 U 1 1 57E15580
 P 4400 4425
@@
 $EndComp
 $Comp
-L Led_Small D?
+L Wiring-Diagram-v2-rescue:Led_Small D?
 U 1 1 57E155BC
 P 4400 5525
@@
 $EndComp
 $Comp
-L SW_NO SW8
+L Supermileage:SW_NO SW8
 U 1 1 57E15EB3
 P 6150 5325
@@
 $EndComp
 $Comp
-L R R?
+L Device:R R?
 U 1 1 57E1710F
 P 4850 5525
@@
 $EndComp
 $Comp
-L R R?
+L Device:R R?
 U 1 1 57E17292
 P 4850 4775
@@
 $EndComp
 $Comp
-L R R?
+L Device:R R?
 U 1 1 57E172E2
 P 4850 5075
@@
 $EndComp
 $Comp
-L R R?
+L Device:R R?
 U 1 1 57E17343
 P 4850 4425
@@
 GND
 $Comp
-L SW_SPST SW4
+L Supermileage:SW_SPST SW4
 U 1 1 57E14E5E
 P 3550 5525
@@
 	3150 6575 3350 6575
 Wire Wire Line
-	3750 5525 4300 5525
+	3750 5525 4000 5525
 Wire Wire Line
 	4000 6075 3750 6075
@@
 	5850 4925 5850 5325
 Wire Wire Line
-	4000 5325 5950 5325
+	4000 5325 5850 5325
 Connection ~ 5850 5325
 Wire Wire Line
 	6350 4925 6450 4925
 Wire Wire Line
-	6450 4925 6450 7325
+	6450 4925 6450 5325
 Wire Wire Line
 	6450 5325 6350 5325
@@
 	5450 5525 5000 5525
 Wire Wire Line
-	4000 5525 4000 6925
-Wire Wire Line
-	3150 5075 4300 5075
+	4000 5525 4000 6075
+Wire Wire Line
+	3150 5075 4000 5075
 Wire Wire Line
 	4300 4775 3150 4775
@@
 	5450 7125 3150 7125
 Wire Wire Line
-	5450 3975 5450 7125
+	5450 3975 5450 4425
 Wire Wire Line
 	6450 7325 3150 7325
@@
 	4000 5325 4000 5075
 Connection ~ 4000 5075
+Wire Wire Line
+	5450 5075 5450 5525
+Wire Wire Line
+	5450 4775 5450 5075
+Wire Wire Line
+	5450 4425 5450 4775
+Wire Wire Line
+	4000 5525 4300 5525
+Wire Wire Line
+	4000 6075 4000 6575
+Wire Wire Line
+	5850 5325 5950 5325
+Wire Wire Line
+	6450 5325 6450 7325
+Wire Wire Line
+	4000 6575 4000 6925
+Wire Wire Line
+	5450 5525 5450 7125
+Wire Wire Line
+	4000 5075 4300 5075
 $EndSCHEMATC
