File: Sting/schematics/StingSchematics.sch (KiCad schematic (older format))
At the start: 30 parts, among them M1 Starter Motor, SW1 Master Power, SW2 Key, SW3 External, SW4 Driver, SW5 Engine Start, SW5 Horn, SW6 Engine Stop, SW6 Horn, SW7 O2 Switch

Commit message: Filled in the Back_Of_Car page more.
Connections:
- net labels added: System_V
- wire segments 92 -> 93
Changed lines of the file:
@@
 Wire Wire Line
 	4650 7100 4750 7100
+Text GLabel 1600 1450 2    60   Output ~ 0
+System_V
+Wire Wire Line
+	1600 1450 1500 1450
+Connection ~ 1500 1450
 $EndSCHEMATC

Commit message: Added fuse before other components.
Parts:
- added F?: 20A, symbol FUSE
- renumbered SW5 to SW7, SW6 to SW8, SW7 to SW9
Connections:
- wire segments 93 -> 94
Other:
- moved on the sheet: CR1B, M1
Changed lines of the file:
@@
 L CR CR1
 U 2 1 57460537
-P 5900 1450
-F 0 "CR1" H 5900 1275 60  0000 C CNN
-F 1 "Starter" H 5900 1600 60  0000 C CNN
-F 2 "" H 5900 1450 60  0000 C CNN
-F 3 "" H 5900 1450 60  0000 C CNN
-	2    5900 1450
+P 5900 1650
+F 0 "CR1" H 5900 1475 60  0000 C CNN
+F 1 "Starter" H 5900 1800 60  0000 C CNN
+F 2 "" H 5900 1650 60  0000 C CNN
+F 3 "" H 5900 1650 60  0000 C CNN
+	2    5900 1650
 	1    0    0    -1
 $EndComp
@@
 $EndComp
 $Comp
-L SW_NO SW5
+L SW_NO SW7
 U 1 1 574B8E3A
 P 2600 4500
-F 0 "SW5" H 2725 4650 60  0000 C CNN
+F 0 "SW7" H 2725 4650 60  0000 C CNN
 F 1 "Horn" H 2600 4400 60  0000 C CNN
 F 2 "" H 2600 4500 60  0000 C CNN
@@
 $EndComp
 $Comp
-L SW_NO SW6
+L SW_NO SW8
 U 1 1 574B8F31
 P 2600 4900
-F 0 "SW6" H 2725 5050 60  0000 C CNN
+F 0 "SW8" H 2725 5050 60  0000 C CNN
 F 1 "Horn" H 2600 4800 60  0000 C CNN
 F 2 "" H 2600 4900 60  0000 C CNN
@@
 	1    0    0    -1
 $EndComp
-Wire Wire Line
-	2750 1100 6400 1100
 Wire Wire Line
 	2000 1100 2350 1100
@@
 $EndComp
 $Comp
-L SW_SPDT SW7
+L SW_SPDT SW9
 U 1 1 574BE58C
 P 3550 6650
-F 0 "SW7" H 3550 6550 60  0000 C CNN
+F 0 "SW9" H 3550 6550 60  0000 C CNN
 F 1 "O2 Switch" H 3550 6900 60  0000 C CNN
 F 2 "" H 3550 6650 60  0000 C CNN
@@
 $EndComp
 Wire Wire Line
-	5750 1450 5500 1450
-Wire Wire Line
-	5500 1450 5500 1100
+	5750 1650 5500 1650
+Wire Wire Line
+	5500 1650 5500 1100
 Connection ~ 5500 1100
 $Comp
 L Motor M1
 U 1 1 57A0B372
-P 6550 1450
-F 0 "M1" H 6550 1450 60  0000 C CNN
-F 1 "Starter Motor" H 6550 1250 60  0000 C CNN
-F 2 "" H 6550 1450 60  0000 C CNN
-F 3 "" H 6550 1450 60  0000 C CNN
-F 4 "Mouser" H 6550 1450 60  0001 C CNN "Distributor"
-	1    6550 1450
-	1    0    0    -1
-$EndComp
-Wire Wire Line
-	6250 1450 6050 1450
-Wire Wire Line
-	7200 1450 6850 1450
-Connection ~ 7200 1450
+P 6550 1650
+F 0 "M1" H 6550 1650 60  0000 C CNN
+F 1 "Starter Motor" H 6550 1450 60  0000 C CNN
+F 2 "" H 6550 1650 60  0000 C CNN
+F 3 "" H 6550 1650 60  0000 C CNN
+F 4 "Mouser" H 6550 1650 60  0001 C CNN "Distributor"
+	1    6550 1650
+	1    0    0    -1
+$EndComp
+Wire Wire Line
+	6250 1650 6050 1650
+Wire Wire Line
+	7200 1650 6850 1650
+Connection ~ 7200 1650
 $Sheet
 S 1032 9218 2418 1082
@@
 	1600 1450 1500 1450
 Connection ~ 1500 1450
+$Comp
+L FUSE F?
+U 1 1 586EB9BF
+P 5950 1100
+F 0 "F?" H 6050 1150 50  0001 C CNN
+F 1 "20A" H 5950 1250 50  0000 C CNN
+F 2 "" H 5950 1100 50  0000 C CNN
+F 3 "" H 5950 1100 50  0000 C CNN
+	1    5950 1100
+	1    0    0    -1
+$EndComp
+Wire Wire Line
+	2750 1100 5700 1100
+Wire Wire Line
+	6200 1100 6400 1100
 $EndSCHEMATC

Commit message: added a relay to enable the starter relay
Parts:
- added CR1: CR, symbol CR
- BT?: symbol Battery -> Battery-RESCUE-StingSchematics
- D? (x4): symbol LED -> LED-RESCUE-StingSchematics
- renumbered CR1 to CR4
Connections:
- net labels added: Starter
- wire segments 94 -> 132
Other:
- moved on the sheet: CB3, CR2B, CR4A, SW7, SW8, SW9

Commit message: added things, namely edited EFI_BREAKOUT
Parts:
- BT?: symbol Battery-RESCUE-StingSchematics -> StingSchematics-rescue:Battery-RESCUE-StingSchematics
- CB1, CB2, CB3: symbol CB -> Supermileage:CB
- CR1, CR3, CR4: symbol CR -> Supermileage:CR
- CR2: symbol 4P_Relay -> Supermileage:4P_Relay
- D?: symbol D -> StingSchematics-rescue:D
- D? (x4): symbol LED-RESCUE-StingSchematics -> StingSchematics-rescue:LED-RESCUE-StingSchematics
- F?: symbol FUSE -> StingSchematics-rescue:FUSE
- L?: symbol Fuel_Injector -> Supermileage:Fuel_Injector
- M1: symbol Motor -> Supermileage:Motor
- R? (x3): symbol R -> StingSchematics-rescue:R
- SP?: symbol Horn -> Supermileage:Horn
- SW1, SW2, SW3, SW4: symbol SW_SPST -> Supermileage:SW_SPST
- SW5, SW6, SW7, SW8: symbol SW_NO -> Supermileage:SW_NO
- SW9: symbol SW_SPDT -> Supermileage:SW_SPDT
- U?: symbol O2_Sensor -> Supermileage:O2_Sensor
- U?: symbol RPM_Sensor -> Supermileage:RPM_Sensor
- U?: symbol Ignition -> Supermileage:Ignition
Changed lines of the file:
@@
-EESchema Schematic File Version 2
-LIBS:StingSchematics-rescue
-LIBS:power
-LIBS:device
-LIBS:transistors
-LIBS:conn
-LIBS:linear
-LIBS:regul
-LIBS:74xx
-LIBS:cmos4000
-LIBS:adc-dac
-LIBS:memory
-LIBS:xilinx
-LIBS:microcontrollers
-LIBS:dsp
-LIBS:microchip
-LIBS:analog_switches
-LIBS:motorola
-LIBS:texas
-LIBS:intel
-LIBS:audio
-LIBS:interface
-LIBS:digital-audio
-LIBS:philips
-LIBS:display
-LIBS:cypress
-LIBS:siliconi
-LIBS:opto
-LIBS:atmel
-LIBS:contrib
-LIBS:valves
-LIBS:Supermileage
-LIBS:relays_switches
+EESchema Schematic File Version 4
 LIBS:StingSchematics-cache
-EELAYER 25 0
+EELAYER 26 0
 EELAYER END
 $Descr USLetter 8500 11000 portrait
@@
 $EndDescr
 $Comp
-L Battery-RESCUE-StingSchematics BT?
+L StingSchematics-rescue:Battery-RESCUE-StingSchematics BT?
 U 1 1 5745DF94
 P 6550 1100
@@
 $EndComp
 $Comp
-L +12V #PWR?
+L power:+12V #PWR?
 U 1 1 5745E309
 P 1500 900
@@
 $EndComp
 $Comp
-L CB CB1
+L Supermileage:CB CB1
 U 1 1 5745EB4B
 P 1850 1100
@@
 $EndComp
 $Comp
-L CB CB2
+L Supermileage:CB CB2
 U 1 1 5745ECAF
 P 1850 2900
@@
 $EndComp
 $Comp
-L CB CB3
+L Supermileage:CB CB3
 U 1 1 5745ED2E
 P 1850 6450
@@
 $EndComp
 $Comp
-L SW_SPST SW1
+L Supermileage:SW_SPST SW1
 U 1 1 5745EFDC
 P 2550 1100
@@
 $EndComp
 $Comp
-L SW_SPST SW2
+L Supermileage:SW_SPST SW2
 U 1 1 5745F17B
 P 2550 2900
@@
 $EndComp
 $Comp
-L SW_SPST SW3
+L Supermileage:SW_SPST SW3
 U 1 1 5745F1FD
 P 3100 2900
@@
 $EndComp
 $Comp
-L SW_SPST SW4
+L Supermileage:SW_SPST SW4
 U 1 1 5745F230
 P 3650 2900
@@
 $EndComp
 $Comp
-L SW_NO SW5
+L Supermileage:SW_NO SW5
 U 1 1 5745FA2B
 P 4800 2900
@@
 $EndComp
 $Comp
-L CR CR4
+L Supermileage:CR CR4
 U 1 1 574604CA
 P 6700 4700
@@
 $EndComp
 $Comp
-L CR CR4
+L Supermileage:CR CR4
 U 2 1 57460537
 P 5900 1650
@@
 $EndComp
 $Comp
-L D D?
+L StingSchematics-rescue:D D?
 U 1 1 574B62AD
 P 6050 3300
@@
 $EndComp
 $Comp
-L LED-RESCUE-StingSchematics D?
+L StingSchematics-rescue:LED-RESCUE-StingSchematics D?
 U 1 1 574B6632
 P 6700 3350
@@
 $EndComp
 $Comp
-L CR CR3
+L Supermileage:CR CR3
 U 1 1 574B6FFB
 P 6700 4200
@@
 $EndComp
 $Comp
-L CR CR3
+L Supermileage:CR CR3
 U 3 1 574B710A
 P 4800 3700
@@
 $EndComp
 $Comp
-L SW_NO SW6
+L Supermileage:SW_NO SW6
 U 1 1 574B71D3
 P 4800 4200
@@
 $EndComp
 $Comp
-L SW_NO SW7
+L Supermileage:SW_NO SW7
 U 1 1 574B8E3A
 P 2600 5100
@@
 $EndComp
 $Comp
-L SW_NO SW8
+L Supermileage:SW_NO SW8
 U 1 1 574B8F31
 P 2600 5500
@@
 Connection ~ 7200 5500
 $Comp
-L LED-RESCUE-StingSchematics D?
+L StingSchematics-rescue:LED-RESCUE-StingSchematics D?
 U 1 1 574BA137
 P 5600 2600
@@
 $EndComp
 $Comp
-L LED-RESCUE-StingSchematics D?
+L StingSchematics-rescue:LED-RESCUE-StingSchematics D?
 U 1 1 574BA223
 P 5200 2400
@@
 $EndComp
 $Comp
-L R R?
+L StingSchematics-rescue:R R?
 U 1 1 574BA2CD
 P 6000 2600
@@
 $EndComp
 $Comp
-L R R?
+L StingSchematics-rescue:R R?
 U 1 1 574BA322
 P 6000 2400
@@
 Connection ~ 3100 5500
 $Comp
-L LED-RESCUE-StingSchematics D?
+L StingSchematics-rescue:LED-RESCUE-StingSchematics D?
 U 1 1 574BCF95
 P 6200 6150
@@
 $EndComp
 $Comp
-L R R?
+L StingSchematics-rescue:R R?
 U 1 1 574BD060
 P 6650 6150
@@
 $EndComp
 $Comp
-L SW_SPDT SW9
+L Supermileage:SW_SPDT SW9
 U 1 1 574BE58C
 P 3550 7050
@@
 $EndComp
 $Comp
-L O2_Sensor U?
+L Supermileage:O2_Sensor U?
 U 1 1 574BF13D
 P 6850 8200
@@
 Connection ~ 7200 6450
 $Comp
-L RPM_Sensor U?
+L Supermileage:RPM_Sensor U?
 U 1 1 574C7D55
 P 6850 7650
@@
 	6300 7800 6300 7400
 $Comp
-L Fuel_Injector L?
+L Supermileage:Fuel_Injector L?
 U 1 1 574C922C
 P 6850 6750
@@
 	5750 6800 6550 6800
 $Comp
-L Ignition U?
+L Supermileage:Ignition U?
 U 1 1 574CABB8
 P 6850 7200
@@
 $EndComp
 $Comp
-L GND #PWR?
+L power:GND #PWR?
 U 1 1 574CD77C
 P 7200 8850
@@
 $EndComp
 $Comp
-L Horn SP?
+L Supermileage:Horn SP?
 U 1 1 574CF991
 P 6700 5500
@@
 $EndSheet
 $Comp
-L +12V #PWR?
+L power:+12V #PWR?
 U 1 1 574D131E
 P 1500 8850
@@
 $EndComp
 $Comp
-L 4P_Relay CR2
+L Supermileage:4P_Relay CR2
 U 1 1 57A033A7
 P 6700 3700
@@
 $EndComp
 $Comp
-L 4P_Relay CR2
+L Supermileage:4P_Relay CR2
 U 2 1 57A034BE
 P 2550 6450
@@
 $EndComp
 $Comp
-L 4P_Relay CR2
+L Supermileage:4P_Relay CR2
 U 4 1 57A04179
 P 5400 3700
@@
 Connection ~ 5500 1100
 $Comp
-L Motor M1
+L Supermileage:Motor M1
 U 1 1 57A0B372
 P 6550 1650
@@
 System_V
 $Comp
-L FUSE F?
+L StingSchematics-rescue:FUSE F?
 U 1 1 586EB9BF
 P 5950 1100
@@
 Connection ~ 1500 1450
 $Comp
-L CR CR1
+L Supermileage:CR CR1
 U 2 1 59D15580
 P 5400 4700
@@
 $EndComp
 $Comp
-L CR CR1
+L Supermileage:CR CR1
 U 1 1 59D156BB
 P 6700 2900
